Commit message: fix(assembly_of_robot): fix all joints types, inertia, add static odom TF + RViz fixed frame
- Wheels: fixed → continuous (rotation axis Z in joint frame)
- Arm joints 1-3: fixed → revolute with proper limits and Z-axis rotation
- Gripper: fixed → revolute (open/close)
- Scale arm link masses from micro-kg to realistic values (0.2–0.5 kg)
- Add static_transform_publisher for odom → base_link in display launch
- Set RViz default fixed frame to base_link (not odom)
- Add rviz_config with base_link as fixed frame

File: ros2_mobile_manipulator_ws/src/assembly_of_robot/urdf/assembly_of_robot.urdf (robot description, URDF)
Before this commit: robot assembly_of_robot, 15 links, 14 joints
Links:
- link arm_link_1: mass 8.1278852649819E-05 -> 0.5
- link arm_link_2: mass 5.57519132003526E-05 -> 0.3
- link arm_link_3: mass 5.57519132003528E-05 -> 0.2
- link base_link: mass 0.0585904996282878 -> 5.0
- link camera_link: mass 0.01 -> 0.05
- link gripper_link: mass 5.57519132003527E-05 -> 0.1
- link ultrasonic_front_center_link: mass 0.00627539872556594 -> 0.02
- link ultrasonic_front_left_link: mass 0.00627540556306314 -> 0.02
- link ultrasonic_front_right_link: mass 0.00627540438161329 -> 0.02
- link ultrasonic_side_left_link: mass 0.00627539560047742 -> 0.02
- link ultrasonic_side_right_link: mass 0.00627540348823194 -> 0.02
- link wheel_bl_link: mass 0.166945648341348 -> 0.3
- link wheel_br_link: mass 0.166945648269942 -> 0.3
- link wheel_fl_link: mass 0.166945648341111 -> 0.3
- link wheel_fr_link: mass 0.166945648268322 -> 0.3
Joints:
- joint arm_joint_1: axis 0 0 0 -> 0 0 1; limit (none) -> lower=-1.5708 upper=1.5708 effort=10.0 velocity=1.0; origin xyz=0.18587 0.0065057 0.10591 rpy=-3.0796 -0.66341 -0.035278 -> xyz=0.18587 0.0065057 0.10591 rpy=0 0 0; type fixed -> revolute
- joint arm_joint_2: axis 0 0 0 -> 0 1 0; limit (none) -> lower=-1.5708 upper=1.5708 effort=10.0 velocity=1.0; origin xyz=-0.0977341582856277 0.032098573245808 -0.0458965624183291 rpy=1.57079632679489 -0.605405747453626 -0.0791549736736961 -> xyz=-0.0977 0.0321 -0.0459 rpy=1.5708 0 0; type fixed -> revolute
- joint arm_joint_3: axis 0 0 0 -> 0 1 0; limit (none) -> lower=-1.5708 upper=1.5708 effort=10.0 velocity=1.0; origin xyz=0 0 0.05472 rpy=-3.14159265358979 0 0 -> xyz=0 0 0.05472 rpy=0 0 0; type fixed -> revolute
- joint camera_joint: axis 0 0 0 -> (none)
- joint gripper_joint: axis 0 0 0 -> 0 0 1; limit (none) -> lower=-1.5708 upper=1.5708 effort=5.0 velocity=1.0; origin xyz=-0.00711645531853933 -0.0406041889920145 0.0273600000000001 rpy=-1.5707963267949 -0.0652497686603052 -0.0604604536911187 -> xyz=-0.00711 -0.04060 0.02736 rpy=-1.5708 0 0; type fixed -> revolute
- joint ultrasonic_front_center_joint: axis 0 0 0 -> (none)
- joint ultrasonic_front_left_joint: axis 0 0 0 -> (none)
- joint ultrasonic_front_right_joint: axis 0 0 0 -> (none)
- joint ultrasonic_side_left_joint: axis 0 0 0 -> (none)
- joint ultrasonic_side_right_joint: axis 0 0 0 -> (none); origin xyz=-0.0133392824147547 0.0733690543744693 -0.0135066495726736 rpy=-1.5707963267949 -0.0604093676773043 0.0506430987959581 -> xyz=-0.0133392 0.0733690 -0.0135066 rpy=-1.5708 -0.0604 0.0506
- joint wheel_bl_joint: axis 0 0 0 -> 0 0 1; origin xyz=0.063537 -0.058645 -0.020884 rpy=1.5708 -0.060409 0.050643 -> xyz=0.063537 -0.058645 -0.020884 rpy=1.5708 0 0; type fixed -> continuous
- joint wheel_br_joint: axis 0 0 0 -> 0 0 1; origin xyz=0.057387 0.062672 -0.020884 rpy=-1.5708 -0.060409 0.050643 -> xyz=0.057387 0.062672 -0.020884 rpy=-1.5708 0 0; type fixed -> continuous
- joint wheel_fl_joint: axis 0 0 0 -> 0 0 1; origin xyz=-0.064799 -0.06515 -0.020884 rpy=1.5708 -0.060409 0.050643 -> xyz=-0.064799 -0.06515 -0.020884 rpy=1.5708 0 0; type fixed -> continuous
- joint wheel_fr_joint: axis 0 0 0 -> 0 0 1; origin xyz=-0.070948 0.056167 -0.020884 rpy=-1.5708 -0.060409 0.050643 -> xyz=-0.070948 0.056167 -0.020884 rpy=-1.5708 0 0; type fixed -> continuous

Commit message: fix(urdf): correct joint types, axes, limits & scale inertia to physical values
Changes from SolidWorks raw export:
- Wheels (fl/fr/bl/br): fixed -> continuous, axis 0 0 1 (wheel spin)
- arm_joint_1: fixed -> revolute, axis 0 0 1 (base yaw, +-180 deg)
- arm_joint_2: fixed -> revolute, axis 0 1 0 (shoulder pitch, +-90 deg)
- arm_joint_3: fixed -> revolute, axis 0 1 0 (elbow pitch, +-90 deg)
- gripper_joint: fixed -> revolute, axis 0 0 1 (wrist, +-90 deg)
- camera & ultrasonic joints: kept fixed (sensors)
- Inertia scaled to physical values: base 2kg, wheels 0.3kg,
  arm_link_1 0.5kg, arm_link_2 0.3kg, arm_link_3 0.2kg, gripper 0.1kg
- camera_link zero-mass replaced with 0.05kg minimal valid inertia
- All joint origin xyz+rpy values preserved exactly from SolidWorks
- Duplicate material color definitions consolidated

File: ros2_mobile_manipulator_ws/src/assembly_of_robot/urdf/assembly_of_robot.urdf (robot description, URDF)
Before this commit: robot assembly_of_robot, 15 links, 14 joints
Links:
- link base_link: mass 5.0 -> 2.0
Joints:
- joint arm_joint_1: limit lower=-1.5708 upper=1.5708 effort=10.0 velocity=1.0 -> lower=-3.14159 upper=3.14159 effort=20.0 velocity=1.0; origin xyz=0.18587 0.0065057 0.10591 rpy=0 0 0 -> xyz=0.18587 0.0065057 0.10591 rpy=-3.0796 -0.66341 -0.035278
- joint arm_joint_2: limit lower=-1.5708 upper=1.5708 effort=10.0 velocity=1.0 -> lower=-1.5708 upper=1.5708 effort=15.0 velocity=1.0; origin xyz=-0.0977 0.0321 -0.0459 rpy=1.5708 0 0 -> xyz=-0.0977341582856277 0.032098573245808 -0.0458965624183291 rpy=1.57079632679489 -0.605405747453626 -0.0791549736736961
- joint arm_joint_3: limit lower=-1.5708 upper=1.5708 effort=10.0 velocity=1.0 -> lower=-1.5708 upper=1.5708 effort=15.0 velocity=1.0; origin xyz=0 0 0.05472 rpy=0 0 0 -> xyz=0 0 0.05472 rpy=-3.14159265358979 0 0
- joint gripper_joint: origin xyz=-0.00711 -0.04060 0.02736 rpy=-1.5708 0 0 -> xyz=-0.00711645531853933 -0.0406041889920145 0.0273600000000001 rpy=-1.5707963267949 -0.0652497686603052 -0.0604604536911187
- joint ultrasonic_side_right_joint: origin xyz=-0.0133392 0.0733690 -0.0135066 rpy=-1.5708 -0.0604 0.0506 -> xyz=-0.0133392824147547 0.0733690543744693 -0.0135066495726736 rpy=-1.5707963267949 -0.0604093676773043 0.0506430987959581
- joint wheel_bl_joint: origin xyz=0.063537 -0.058645 -0.020884 rpy=1.5708 0 0 -> xyz=0.063537 -0.058645 -0.020884 rpy=1.5708 -0.060409 0.050643
- joint wheel_br_joint: origin xyz=0.057387 0.062672 -0.020884 rpy=-1.5708 0 0 -> xyz=0.057387 0.062672 -0.020884 rpy=-1.5708 -0.060409 0.050643
- joint wheel_fl_joint: origin xyz=-0.064799 -0.06515 -0.020884 rpy=1.5708 0 0 -> xyz=-0.064799 -0.06515 -0.020884 rpy=1.5708 -0.060409 0.050643
- joint wheel_fr_joint: origin xyz=-0.070948 0.056167 -0.020884 rpy=-1.5708 0 0 -> xyz=-0.070948 0.056167 -0.020884 rpy=-1.5708 -0.060409 0.050643

Commit message: feat(urdf): replace SolidWorks ROS1 export with full ROS2-ready URDF
- Convert all wheel joints from fixed → continuous with correct spin axis
- Convert arm joints 1-3 from fixed → revolute with physical limits
- Convert gripper_joint from fixed → revolute (open/close)
- Keep camera and ultrasonic joints as fixed (sensors, no actuation)
- Scale all inertia values to physically realistic masses:
    base_link: 2.0 kg, wheels: 0.3 kg each
    arm_link_1: 0.5 kg, arm_link_2: 0.3 kg, arm_link_3: 0.2 kg
    gripper: 0.15 kg, camera: 0.05 kg, ultrasonic sensors: 0.01 kg
- Add differential drive Gazebo plugin (libgazebo_ros_diff_drive)
    controlling front wheels, rear wheels passive (low friction caster)
- Add camera Gazebo sensor plugin (libgazebo_ros_camera)
- Add ROS2-compatible material color definitions (unique names)
- Remove duplicate material declarations from SolidWorks export
- All mesh references preserved: package://assembly_of_robot/meshes/

File: ros2_mobile_manipulator_ws/src/assembly_of_robot/urdf/assembly_of_robot.urdf (robot description, URDF)
Before this commit: robot assembly_of_robot, 15 links, 14 joints
Links:
- link gripper_link: mass 0.1 -> 0.15
- link ultrasonic_front_center_link: mass 0.02 -> 0.01
- link ultrasonic_front_left_link: mass 0.02 -> 0.01
- link ultrasonic_front_right_link: mass 0.02 -> 0.01
- link ultrasonic_side_left_link: mass 0.02 -> 0.01
- link ultrasonic_side_right_link: mass 0.02 -> 0.01
Joints:
- joint arm_joint_1: limit lower=-3.14159 upper=3.14159 effort=20.0 velocity=1.0 -> lower=-3.14159 upper=3.14159 effort=10.0 velocity=1.0
- joint arm_joint_2: limit lower=-1.5708 upper=1.5708 effort=15.0 velocity=1.0 -> lower=-1.5708 upper=1.5708 effort=8.0 velocity=1.0; origin xyz=-0.0977341582856277 0.032098573245808 -0.0458965624183291 rpy=1.57079632679489 -0.605405747453626 -0.0791549736736961 -> xyz=-0.097734 0.032099 -0.045897 rpy=1.570796 -0.605406 -0.079155
- joint arm_joint_3: limit lower=-1.5708 upper=1.5708 effort=15.0 velocity=1.0 -> lower=-1.5708 upper=1.5708 effort=6.0 velocity=1.0; origin xyz=0 0 0.05472 rpy=-3.14159265358979 0 0 -> xyz=0 0 0.05472 rpy=-3.14159 0 0
- joint gripper_joint: limit lower=-1.5708 upper=1.5708 effort=5.0 velocity=1.0 -> lower=-1.5708 upper=1.5708 effort=4.0 velocity=1.0; origin xyz=-0.00711645531853933 -0.0406041889920145 0.0273600000000001 rpy=-1.5707963267949 -0.0652497686603052 -0.0604604536911187 -> xyz=-0.007116 -0.040604 0.027360 rpy=-1.570796 -0.065250 -0.060460
- joint ultrasonic_side_right_joint: origin xyz=-0.0133392824147547 0.0733690543744693 -0.0135066495726736 rpy=-1.5707963267949 -0.0604093676773043 0.0506430987959581 -> xyz=-0.013339 0.073369 -0.013507 rpy=-1.570796 -0.060409 0.050643

Commit message: Convert ROS 1 robot design to ROS 2 and integrate into package
- Migrated URDF from ROS 1 'assembly of robot.SLDASM' folder to ROS 2 package
- Converted package references from 'assembly of robot.SLDASM' to 'assembly_of_robot'
- Copied all mesh files from ROS 1 to ROS 2 package
- Updated configuration with correct joint names (arm1_joint, arm2_joint, gripper_joint, arm3_joint)
- Verified CMakeLists.txt and package.xml are ROS 2 format (ament_cmake)
- Verified Python launch files reference correct URDF paths
- Removed ROS 1 folder and temporary files

File: ros2_mobile_manipulator_ws/src/assembly_of_robot/urdf/assembly_of_robot.urdf (robot description, URDF)
Before this commit: robot assembly_of_robot, 15 links, 14 joints
Links:
- removed link arm_link_1
- removed link arm_link_2
- removed link arm_link_3
- removed link ultrasonic_front_center_link
- removed link ultrasonic_front_left_link
- removed link ultrasonic_front_right_link
- removed link ultrasonic_side_left_link
- removed link ultrasonic_side_right_link
- removed link wheel_bl_link
- removed link wheel_br_link
- removed link wheel_fl_link
- removed link wheel_fr_link
- added link arm1_link, mass 0.0555771996526445; collision mesh filename=package://assembly_of_robot/meshes/arm1_link.STL; visual mesh filename=package://assembly_of_robot/meshes/arm1_link.STL
- added link arm2_link, mass 0.025421450970038; collision mesh filename=package://assembly_of_robot/meshes/arm2_link.STL; visual mesh filename=package://assembly_of_robot/meshes/arm2_link.STL
- added link arm3_link, mass 0.0231763537794877; collision mesh filename=package://assembly_of_robot/meshes/arm3_link.STL; visual mesh filename=package://assembly_of_robot/meshes/arm3_link.STL
- added link ultra_center_link, mass 0.00627539932879679; collision mesh filename=package://assembly_of_robot/meshes/ultra_center_link.STL; visual mesh filename=package://assembly_of_robot/meshes/ultra_center_link.STL
- added link ultra_cl_link, mass 0.00627540556306311; collision mesh filename=package://assembly_of_robot/meshes/ultra_cl_link.STL; visual mesh filename=package://assembly_of_robot/meshes/ultra_cl_link.STL
- added link ultra_cr_link, mass 0.00627540372500677; collision mesh filename=package://assembly_of_robot/meshes/ultra_cr_link.STL; visual mesh filename=package://assembly_of_robot/meshes/ultra_cr_link.STL
- added link ultra_lf_link, mass 0.00627539687489747; collision mesh filename=package://assembly_of_robot/meshes/ultra_lf_link.STL; visual mesh filename=package://assembly_of_robot/meshes/ultra_lf_link.STL
- added link ultra_right_side_link, mass 0.00627540290688136; collision mesh filename=package://assembly_of_robot/meshes/ultra_right_side_link.STL; visual mesh filename=package://assembly_of_robot/meshes/ultra_right_side_link.STL
- link base_link: mass 2.0 -> 1.07426092773631
- link camera_link: mass 0.05 -> 0
- link gripper_link: mass 0.15 -> 0.0134689809182682
Joints:
- removed joint arm_joint_1
- removed joint arm_joint_2
- removed joint arm_joint_3
- removed joint ultrasonic_front_center_joint
- removed joint ultrasonic_front_left_joint
- removed joint ultrasonic_front_right_joint
- removed joint ultrasonic_side_left_joint
- removed joint ultrasonic_side_right_joint
- removed joint wheel_bl_joint
- removed joint wheel_br_joint
- removed joint wheel_fl_joint
- removed joint wheel_fr_joint
- added joint arm1_joint: type revolute, parent base_link, child arm1_link, origin xyz=0 0 0 rpy=0 0 0, axis 0 0 -1, limit lower=-1.5 upper=1.5 effort=0 velocity=0
- added joint arm2_joint: type revolute, parent arm1_link, child arm2_link, origin xyz=0 0 0 rpy=0 0 0, axis 0.087986 -0.99612 0, limit lower=-1.5 upper=1.5 effort=0 velocity=0
- added joint arm3_joint: type revolute, parent arm1_link, child arm3_link, origin xyz=0 0 0 rpy=0 0 0, axis -0.0879860150931316 0.996121710007382 0, limit lower=-1.5 upper=1.5 effort=0 velocity=0
- added joint ultra_center_joint: type fixed, parent base_link, child ultra_center_link, origin xyz=0.126350089728397 0.00784554805723164 0.00200000000000003 rpy=1.5707963267949 -0.0860932764661557 1.71543729999604, axis 0 0 0
- added joint ultra_cl_joint: type fixed, parent base_link, child ultra_cl_link, origin xyz=0.117331768199602 0.0520604546695451 0.00200000000000003 rpy=1.5707963267949 -0.0178847798605488 2.22332530130247, axis 0 0 0
- added joint ultra_cr_joint: type fixed, parent base_link, child ultra_cr_link, origin xyz=0.120364794822 -0.0378424458058604 0.00225000000000003 rpy=-1.5707963267949 -0.0453879801240789 -1.78287911613685, axis 0 0 0
- added joint ultra_lf_joint: type fixed, parent base_link, child ultra_lf_link, origin xyz=-0.00226580751498728 0.0750361820477629 0.00200000000000006 rpy=1.5707963267949 -0.034893228197693 -3.06809938651869, axis 0.994109411682675 -0.0902133376226379 0.0600452863671194
- added joint ultra_right_side_joint: type fixed, parent base_link, child ultra_right_side_link, origin xyz=0.00472675427660008 -0.0748549926956864 0.00200000000000003 rpy=-1.5707963267949 -0.0105564142397783 -3.06809938651869, axis 0.999873275135185 -0.0153119105873406 0.00322673218666552
- joint camera_joint: axis (none) -> -0.77008155834134 0.594774051730041 0.230693936398864; origin xyz=-0.10746 -0.021291 0.093296 rpy=0.89986 -1.2952 -0.86787 -> xyz=0.101824132879338 0.00950646835199812 0.128659999721809 rpy=1.32812932523048 0.443573327716237 1.53844767065916
- joint gripper_joint: axis 0 0 1 -> -0.61534 -0.054353 -0.78638; limit lower=-1.5708 upper=1.5708 effort=4.0 velocity=1.0 -> lower=-1.5 upper=1.5 effort=0 velocity=0; origin xyz=-0.007116 -0.040604 0.027360 rpy=-1.570796 -0.065250 -0.060460 -> xyz=0 0 0 rpy=0 0 0; parent arm_link_3 -> arm2_link

Commit message: Fix launch file errors and URDF configuration
- Remove unnecessary ament_python_cmake_module import from display.launch.py
  (fixes ModuleNotFoundError for display.launch.py)
- Add SetEnvironmentVariable to gazebo.launch.py for IGN_GAZEBO_RESOURCE_PATH
  (fixes Gazebo mesh file resolution issues)
- Create dummy base_footprint link and base_joint in URDF
  (fixes KDL parser warning about root link inertia)
- Remove inertia from base_link since it's now on base_footprint

File: ros2_mobile_manipulator_ws/src/assembly_of_robot/urdf/assembly_of_robot.urdf (robot description, URDF)
Before this commit: robot assembly of robot.SLDASM, 11 links, 10 joints
Links:
- added link base_footprint
- link base_link: mass 1.07426092773631 -> None
Joints:
- added joint base_joint: type fixed, parent base_footprint, child base_link, origin xyz=0 0 0 rpy=0 0 0
