Commit message: Fix xacro pi warning in simulation URDF
Agent-Logs-Url: https://github.com/ZainAlabidinShbani/Mobile-Manipulator-Simulation-Academic-Project-Journey/sessions/fa2f838a-51a7-408a-8f21-c1ab4fd277cd

Co-authored-by: ZainAlabidinShbani <233742937+ZainAlabidinShbani@users.noreply.github.com>

File: ros2_mobile_manipulator_ws/src/simulation_pkg/urdf/mobile_manipulator.urdf.xacro (robot description, xacro)
@@ -1,5 +1,5 @@
 <?xml version="1.0"?>
 <robot xmlns:xacro="http://www.ros.org/wiki/xacro" name="mobile_manipulator">
-  <xacro:property name="pi" value="3.141592653589793"/>
+  <xacro:property name="pi_val" value="3.141592653589793"/>
   <xacro:property name="base_length" value="0.46"/>
   <xacro:property name="base_width" value="0.38"/>
@@ -25,11 +25,11 @@
   <joint name="camera_joint" type="fixed"><parent link="arm_base_link"/><child link="camera_link"/><origin xyz="0.15 0 0.28" rpy="0 0 0"/></joint>
   <link name="arm_link_1"><visual><geometry><cylinder length="${arm_link1}" radius="0.04"/></geometry><material name="Red"><color rgba="0.8 0.2 0.2 1.0"/></material></visual></link>
-  <joint name="arm_joint_1" type="revolute"><parent link="arm_base_link"/><child link="arm_link_1"/><origin xyz="0 0 0.1" rpy="0 0 0"/><axis xyz="0 0 1"/><limit lower="-${pi}" upper="${pi}" effort="30" velocity="1.5"/></joint>
+  <joint name="arm_joint_1" type="revolute"><parent link="arm_base_link"/><child link="arm_link_1"/><origin xyz="0 0 0.1" rpy="0 0 0"/><axis xyz="0 0 1"/><limit lower="-${pi_val}" upper="${pi_val}" effort="30" velocity="1.5"/></joint>
   <link name="arm_link_2"><visual><origin xyz="${arm_link2/2.0} 0 0"/><geometry><box size="${arm_link2} 0.05 0.05"/></geometry><material name="Green"><color rgba="0.2 0.8 0.3 1.0"/></material></visual></link>
-  <joint name="arm_joint_2" type="revolute"><parent link="arm_link_1"/><child link="arm_link_2"/><origin xyz="0 0 ${arm_link1}" rpy="0 0 0"/><axis xyz="0 1 0"/><limit lower="-${pi/2.0}" upper="${pi/2.0}" effort="25" velocity="1.5"/></joint>
+  <joint name="arm_joint_2" type="revolute"><parent link="arm_link_1"/><child link="arm_link_2"/><origin xyz="0 0 ${arm_link1}" rpy="0 0 0"/><axis xyz="0 1 0"/><limit lower="-${pi_val/2.0}" upper="${pi_val/2.0}" effort="25" velocity="1.5"/></joint>
   <link name="arm_link_3"><visual><origin xyz="${arm_link3/2.0} 0 0"/><geometry><box size="${arm_link3} 0.045 0.045"/></geometry><material name="Yellow"><color rgba="0.9 0.8 0.2 1.0"/></material></visual></link>
-  <joint name="arm_joint_3" type="revolute"><parent link="arm_link_2"/><child link="arm_link_3"/><origin xyz="${arm_link2} 0 0" rpy="0 0 0"/><axis xyz="0 1 0"/><limit lower="-${pi/2.0}" upper="${pi/2.0}" effort="20" velocity="1.5"/></joint>
+  <joint name="arm_joint_3" type="revolute"><parent link="arm_link_2"/><child link="arm_link_3"/><origin xyz="${arm_link2} 0 0" rpy="0 0 0"/><axis xyz="0 1 0"/><limit lower="-${pi_val/2.0}" upper="${pi_val/2.0}" effort="20" velocity="1.5"/></joint>
   <link name="arm_link_4"><visual><origin xyz="${arm_link3} 0 0"/><geometry><box size="${arm_link3} 0.035 0.035"/></geometry><material name="Purple"><color rgba="0.7 0.2 0.8 1.0"/></material></visual></link>
-  <joint name="arm_joint_4" type="revolute"><parent link="arm_link_3"/><child link="arm_link_4"/><origin xyz="${arm_link3} 0 0" rpy="0 0 0"/><axis xyz="0 1 0"/><limit lower="-${pi}" upper="${pi}" effort="15" velocity="2.0"/></joint>
+  <joint name="arm_joint_4" type="revolute"><parent link="arm_link_3"/><child link="arm_link_4"/><origin xyz="${arm_link3} 0 0" rpy="0 0 0"/><axis xyz="0 1 0"/><limit lower="-${pi_val}" upper="${pi_val}" effort="15" velocity="2.0"/></joint>
   <link name="gripper_link"><visual><geometry><box size="0.06 0.02 0.02"/></geometry><material name="Black"><color rgba="0.1 0.1 0.1 1.0"/></material></visual></link>
   <joint name="gripper_joint" type="fixed"><parent link="arm_link_4"/><child link="gripper_link"/><origin xyz="${arm_link3} 0 0" rpy="0 0 0"/></joint>
