Commit message: Refactor pick-and-place world and task manager configuration
- Updated the pick_and_place.world file to simplify the environment setup, reducing the number of models and adjusting poses for the pick and drop tables.
- Modified task_manager.yaml to maintain consistent formatting.
- Cleaned up launch files for the task manager, ensuring proper imports and structure.
- Adjusted package.xml and setup.py for better clarity and consistency in dependencies and configurations.
- Enhanced fsm_task_manager_node.py for improved readability and maintainability, including better handling of robot states and task execution flow.

File: ros2_mobile_manipulator_ws/src/simulation_pkg/urdf/mobile_manipulator.urdf.xacro (robot description, xacro)
@@ -1,43 +1,16 @@
 <?xml version="1.0"?>
 <robot xmlns:xacro="http://www.ros.org/wiki/xacro" name="mobile_manipulator">
-  <!-- ================================================================ -->
-  <!--  PROPERTIES                                                        -->
-  <!-- ================================================================ -->
-  <!-- Base -->
-  <xacro:property name="base_length" value="0.50"/>
-  <xacro:property name="base_width"  value="0.35"/>
+  <!-- PROPERTIES -->
+  <xacro:property name="base_length" value="0.46"/>
+  <xacro:property name="base_width"  value="0.38"/>
   <xacro:property name="base_height" value="0.12"/>
-  <xacro:property name="base_mass"   value="8.0"/>
-  <!-- Wheel -->
-  <xacro:property name="wheel_radius" value="0.06"/>
-  <xacro:property name="wheel_width"  value="0.04"/>
+  <xacro:property name="base_mass"   value="18.0"/>
+  <xacro:property name="wheel_radius" value="0.05"/>
+  <xacro:property name="wheel_width"  value="0.03"/>
   <xacro:property name="wheel_mass"   value="0.5"/>
-  <xacro:property name="wheel_x_off"  value="0.18"/>
-  <xacro:property name="wheel_y_off"  value="0.195"/>
-  <!-- Arm links (DH-compatible lengths) -->
-  <xacro:property name="link1_length" value="0.10"/>  <!-- shoulder rise   -->
-  <xacro:property name="link2_length" value="0.20"/>  <!-- upper arm       -->
-  <xacro:property name="link3_length" value="0.16"/>  <!-- forearm         -->
-  <xacro:property name="link4_length" value="0.10"/>  <!-- wrist           -->
-  <xacro:property name="arm_mass"     value="0.4"/>
-  <!-- Gripper -->
-  <xacro:property name="finger_length" value="0.06"/>
-  <xacro:property name="finger_mass"   value="0.05"/>
-  <!-- Sensors -->
-  <xacro:property name="camera_mass"  value="0.1"/>
-  <xacro:property name="lidar_mass"   value="0.2"/>
-  <!-- ================================================================ -->
-  <!--  MATERIAL DEFINITIONS                                             -->
-  <!-- ================================================================ -->
-  <material name="dark_grey"><color rgba="0.2 0.2 0.2 1.0"/></material>
-  <material name="light_grey"><color rgba="0.7 0.7 0.7 1.0"/></material>
-  <material name="blue"><color rgba="0.1 0.4 0.8 1.0"/></material>
-  <material name="orange"><color rgba="0.9 0.4 0.0 1.0"/></material>
-  <material name="black"><color rgba="0.05 0.05 0.05 1.0"/></material>
-  <material name="white"><color rgba="0.95 0.95 0.95 1.0"/></material>
-  <!-- ================================================================ -->
-  <!--  MACROS                                                           -->
-  <!-- ================================================================ -->
-  <!-- Inertia helpers -->
+  <xacro:property name="arm_link1" value="0.28"/>
+  <xacro:property name="arm_link2" value="0.24"/>
+  <xacro:property name="arm_link3" value="0.14"/>
+  <!-- INERTIA MACROS -->
   <xacro:macro name="box_inertia" params="m l w h">
     <inertial>
@@ -56,10 +29,10 @@
     </inertial>
   </xacro:macro>
-  <!-- Wheel macro (reused for all 4 wheels) -->
-  <xacro:macro name="wheel" params="name x_sign y_sign">
-    <link name="${name}_wheel_link">
+  <!-- WHEEL MACRO -->
+  <xacro:macro name="wheel" params="name x y">
+    <link name="${name}_link">
       <visual>
         <geometry><cylinder radius="${wheel_radius}" length="${wheel_width}"/></geometry>
-        <material name="black"/>
+        <material name="black"><color rgba="0.05 0.05 0.05 1"/></material>
       </visual>
       <collision>
@@ -68,31 +41,13 @@
       <xacro:cylinder_inertia m="${wheel_mass}" r="${wheel_radius}" h="${wheel_width}"/>
     </link>
-    <joint name="${name}_wheel_joint" type="continuous">
+    <joint name="${name}_joint" type="continuous">
       <parent link="base_link"/>
-      <child  link="${name}_wheel_link"/>
-      <origin xyz="${x_sign*wheel_x_off} ${y_sign*wheel_y_off} 0"
-              rpy="${pi/2} 0 0"/>
+      <child  link="${name}_link"/>
+      <origin xyz="${x} ${y} 0" rpy="${pi/2} 0 0"/>
       <axis xyz="0 0 1"/>
       <dynamics damping="0.01" friction="0.1"/>
     </joint>
   </xacro:macro>
-  <!-- Arm link macro -->
-  <xacro:macro name="arm_link" params="name length material">
-    <link name="${name}">
-      <visual>
-        <origin xyz="0 0 ${length/2}" rpy="0 0 0"/>
-        <geometry><box size="0.04 0.04 ${length}"/></geometry>
-        <material name="${material}"/>
-      </visual>
-      <collision>
-        <origin xyz="0 0 ${length/2}" rpy="0 0 0"/>
-        <geometry><box size="0.04 0.04 ${length}"/></geometry>
-      </collision>
-      <xacro:box_inertia m="${arm_mass}" l="0.04" w="0.04" h="${length}"/>
-    </link>
-  </xacro:macro>
-  <!-- ================================================================ -->
-  <!--  BASE FOOTPRINT & BASE LINK                                       -->
-  <!-- ================================================================ -->
+  <!-- BASE FOOTPRINT -->
   <link name="base_footprint"/>
   <joint name="base_footprint_joint" type="fixed">
@@ -101,170 +56,218 @@
     <origin xyz="0 0 ${wheel_radius}" rpy="0 0 0"/>
   </joint>
+  <!-- BASE LINK -->
   <link name="base_link">
     <visual>
-      <geometry>
-        <box size="${base_length} ${base_width} ${base_height}"/>
-      </geometry>
-      <material name="blue"/>
+      <origin xyz="0 0 ${base_height/2}"/>
+      <geometry><box size="${base_length} ${base_width} ${base_height}"/></geometry>
+      <material name="gray"><color rgba="0.6 0.6 0.65 1.0"/></material>
     </visual>
     <collision>
-      <geometry>
-        <box size="${base_length} ${base_width} ${base_height}"/>
-      </geometry>
+      <origin xyz="0 0 ${base_height/2}"/>
+      <geometry><box size="${base_length} ${base_width} ${base_height}"/></geometry>
     </collision>
     <xacro:box_inertia m="${base_mass}" l="${base_length}" w="${base_width}" h="${base_height}"/>
   </link>
-  <!-- ================================================================ -->
-  <!--  WHEELS (4x differential drive)                                   -->
-  <!-- ================================================================ -->
-  <xacro:wheel name="front_left"  x_sign="1"  y_sign="1"/>
-  <xacro:wheel name="front_right" x_sign="1"  y_sign="-1"/>
-  <xacro:wheel name="rear_left"   x_sign="-1" y_sign="1"/>
-  <xacro:wheel name="rear_right"  x_sign="-1" y_sign="-1"/>
-  <!-- ================================================================ -->
-  <!--  ARM BASE MOUNT                                                   -->
-  <!-- ================================================================ -->
+  <!-- WHEELS -->
+  <xacro:wheel name="wheel_front_left"  x="0.16"  y="0.21"/>
+  <xacro:wheel name="wheel_front_right" x="0.16"  y="-0.21"/>
+  <xacro:wheel name="wheel_rear_left"   x="-0.16" y="0.21"/>
+  <xacro:wheel name="wheel_rear_right"  x="-0.16" y="-0.21"/>
+  <!-- ARM BASE -->
   <link name="arm_base_link">
     <visual>
-      <geometry><cylinder radius="0.04" length="0.05"/></geometry>
-      <material name="dark_grey"/>
+      <origin xyz="0 0 0.05"/>
+      <geometry><cylinder length="0.1" radius="0.08"/></geometry>
+      <material name="blue"><color rgba="0.2 0.4 0.8 1.0"/></material>
     </visual>
     <collision>
-      <geometry><cylinder radius="0.04" length="0.05"/></geometry>
+      <origin xyz="0 0 0.05"/>
+      <geometry><cylinder length="0.1" radius="0.08"/></geometry>
     </collision>
-    <xacro:cylinder_inertia m="0.3" r="0.04" h="0.05"/>
+    <xacro:cylinder_inertia m="1.0" r="0.08" h="0.1"/>
   </link>
   <joint name="arm_base_joint" type="fixed">
     <parent link="base_link"/>
     <child  link="arm_base_link"/>
-    <origin xyz="0.15 0 ${base_height/2 + 0.025}" rpy="0 0 0"/>
-  </joint>
-  <!-- ================================================================ -->
-  <!--  4-DOF ARM                                                        -->
-  <!-- ================================================================ -->
-  <!-- Joint 1 — Waist (Z rotation) -->
-  <xacro:arm_link name="link1" length="${link1_length}" material="light_grey"/>
-  <joint name="joint1" type="revolute">
-    <parent link="arm_base_link"/>
-    <child  link="link1"/>
-    <origin xyz="0 0 0.025" rpy="0 0 0"/>
-    <axis xyz="0 0 1"/>
-    <limit lower="-3.14159" upper="3.14159" effort="10" velocity="1.0"/>
+    <origin xyz="0 0 0.18" rpy="0 0 0"/>
+  </joint>
+  <!-- ARM LINKS -->
+  <link name="arm_link_1">
+    <visual><geometry><cylinder length="${arm_link1}" radius="0.04"/></geometry>
+      <material name="red"><color rgba="0.8 0.2 0.2 1.0"/></material></visual>
+    <collision><geometry><cylinder length="${arm_link1}" radius="0.04"/></geometry></collision>
+    <xacro:cylinder_inertia m="0.5" r="0.04" h="${arm_link1}"/>
+  </link>
+  <joint name="arm_joint_1" type="revolute">
+    <parent link="arm_base_link"/><child link="arm_link_1"/>
+    <origin xyz="0 0 0.1" rpy="0 0 0"/><axis xyz="0 0 1"/>
+    <limit lower="${-pi}" upper="${pi}" effort="30" velocity="1.5"/>
     <dynamics damping="0.1" friction="0.05"/>
   </joint>
-  <!-- Joint 2 — Shoulder (Y rotation) -->
-  <xacro:arm_link name="link2" length="${link2_length}" material="light_grey"/>
-  <joint name="joint2" type="revolute">
-    <parent link="link1"/>
-    <child  link="link2"/>
-    <origin xyz="0 0 ${link1_length}" rpy="0 0 0"/>
-    <axis xyz="0 1 0"/>
-    <limit lower="-1.5708" upper="1.5708" effort="10" velocity="1.0"/>
+  <link name="arm_link_2">
+    <visual><origin xyz="${arm_link2/2} 0 0"/>
+      <geometry><box size="${arm_link2} 0.05 0.05"/></geometry>
+      <material name="green"><color rgba="0.2 0.8 0.3 1.0"/></material></visual>
+    <collision><origin xyz="${arm_link2/2} 0 0"/>
+      <geometry><box size="${arm_link2} 0.05 0.05"/></geometry></collision>
+    <xacro:box_inertia m="0.4" l="${arm_link2}" w="0.05" h="0.05"/>
+  </link>
+  <joint name="arm_joint_2" type="revolute">
+    <parent link="arm_link_1"/><child link="arm_link_2"/>
+    <origin xyz="0 0 ${arm_link1}" rpy="0 0 0"/><axis xyz="0 1 0"/>
+    <limit lower="${-pi/2}" upper="${pi/2}" effort="25" velocity="1.5"/>
     <dynamics damping="0.1" friction="0.05"/>
   </joint>
-  <!-- Joint 3 — Elbow (Y rotation) -->
-  <xacro:arm_link name="link3" length="${link3_length}" material="light_grey"/>
-  <joint name="joint3" type="revolute">
-    <parent link="link2"/>
-    <child  link="link3"/>
-    <origin xyz="0 0 ${link2_length}" rpy="0 0 0"/>
-    <axis xyz="0 1 0"/>
-    <limit lower="-1.5708" upper="1.5708" effort="8" velocity="1.0"/>
+  <link name="arm_link_3">
+    <visual><origin xyz="${arm_link3/2} 0 0"/>
+      <geometry><box size="${arm_link3} 0.045 0.045"/></geometry>
+      <material name="yellow"><color rgba="0.9 0.8 0.2 1.0"/></material></visual>
+    <collision><origin xyz="${arm_link3/2} 0 0"/>
+      <geometry><box size="${arm_link3} 0.045 0.045"/></geometry></collision>
+    <xacro:box_inertia m="0.3" l="${arm_link3}" w="0.045" h="0.045"/>
+  </link>
+  <joint name="arm_joint_3" type="revolute">
+    <parent link="arm_link_2"/><child link="arm_link_3"/>
+    <origin xyz="${arm_link2} 0 0" rpy="0 0 0"/><axis xyz="0 1 0"/>
+    <limit lower="${-pi/2}" upper="${pi/2}" effort="20" velocity="1.5"/>
     <dynamics damping="0.1" friction="0.05"/>
   </joint>
-  <!-- Joint 4 — Wrist (Y rotation) -->
-  <xacro:arm_link name="link4" length="${link4_length}" material="orange"/>
-  <joint name="joint4" type="revolute">
-    <parent link="link3"/>
-    <child  link="link4"/>
-    <origin xyz="0 0 ${link3_length}" rpy="0 0 0"/>
-    <axis xyz="0 1 0"/>
-    <limit lower="-1.5708" upper="1.5708" effort="5" velocity="1.5"/>
+  <link name="arm_link_4">
+    <visual><origin xyz="${arm_link3} 0 0"/>
+      <geometry><box size="${arm_link3} 0.035 0.035"/></geometry>
+      <material name="purple"><color rgba="0.7 0.2 0.8 1.0"/></material></visual>
+    <collision><origin xyz="${arm_link3} 0 0"/>
+      <geometry><box size="${arm_link3} 0.035 0.035"/></geometry></collision>
+    <xacro:box_inertia m="0.2" l="${arm_link3}" w="0.035" h="0.035"/>
+  </link>
+  <joint name="arm_joint_4" type="revolute">
+    <parent link="arm_link_3"/><child link="arm_link_4"/>
+    <origin xyz="${arm_link3} 0 0" rpy="0 0 0"/><axis xyz="0 1 0"/>
+    <limit lower="${-pi}" upper="${pi}" effort="15" velocity="2.0"/>
     <dynamics damping="0.05" friction="0.02"/>
   </joint>
-  <!-- ================================================================ -->
-  <!--  END EFFECTOR & GRIPPER                                           -->
-  <!-- ================================================================ -->
-  <link name="end_effector_link">
-    <visual>
-      <geometry><sphere radius="0.015"/></geometry>
-      <material name="orange"/>
-    </visual>
-    <inertial>
-      <mass value="0.05"/>
-      <inertia ixx="1e-5" ixy="0" ixz="0" iyy="1e-5" iyz="0" izz="1e-5"/>
-    </inertial>
-  </link>
-  <joint name="end_effector_joint" type="fixed">
-    <parent link="link4"/>
-    <child  link="end_effector_link"/>
-    <origin xyz="0 0 ${link4_length}" rpy="0 0 0"/>
-  </joint>
-  <!-- Left finger -->
+  <!-- GRIPPER -->
+  <link name="gripper_link">
+    <visual><geometry><box size="0.06 0.02 0.02"/></geometry>
+      <material name="black2"><color rgba="0.1 0.1 0.1 1.0"/></material></visual>
+    <collision><geometry><box size="0.06 0.02 0.02"/></geometry></collision>
+    <xacro:box_inertia m="0.1" l="0.06" w="0.02" h="0.02"/>
+  </link>
+  <joint name="gripper_joint" type="fixed">
+    <parent link="arm_link_4"/><child link="gripper_link"/>
+    <origin xyz="${arm_link3} 0 0" rpy="0 0 0"/>
+  </joint>
   <link name="left_finger_link">
-    <visual>
-      <origin xyz="0 0 ${finger_length/2}" rpy="0 0 0"/>
-      <geometry><box size="0.015 0.008 ${finger_length}"/></geometry>
-      <material name="dark_grey"/>
-    </visual>
-    <collision>
-      <origin xyz="0 0 ${finger_length/2}" rpy="0 0 0"/>
-      <geometry><box size="0.015 0.008 ${finger_length}"/></geometry>
-    </collision>
-    <xacro:box_inertia m="${finger_mass}" l="0.015" w="0.008" h="${finger_length}"/>
+    <visual><origin xyz="0.02 0.015 0"/>
+      <geometry><box size="0.04 0.01 0.02"/></geometry>
+      <material name="silver"><color rgba="0.85 0.85 0.85 1.0"/></material></visual>
+    <collision><origin xyz="0.02 0.015 0"/>
+      <geometry><box size="0.04 0.01 0.02"/></geometry></collision>
+    <xacro:box_inertia m="0.05" l="0.04" w="0.01" h="0.02"/>
   </link>
   <joint name="left_finger_joint" type="prismatic">
-    <parent link="end_effector_link"/>
-    <child  link="left_finger_link"/>
-    <origin xyz="0 0.02 0" rpy="0 0 0"/>
-    <axis xyz="0 1 0"/>
-    <limit lower="0.0" upper="0.04" effort="5" velocity="0.1"/>
-  </joint>
-  <!-- Right finger -->
+    <parent link="gripper_link"/><child link="left_finger_link"/>
+    <origin xyz="0.03 0.012 0" rpy="0 0 0"/><axis xyz="0 1 0"/>
+    <limit lower="0.0" upper="0.03" effort="10" velocity="0.5"/>
+  </joint>
   <link name="right_finger_link">
-    <visual>
-      <origin xyz="0 0 ${finger_length/2}" rpy="0 0 0"/>
-      <geometry><box size="0.015 0.008 ${finger_length}"/></geometry>
-      <material name="dark_grey"/>
-    </visual>
-    <collision>
-      <origin xyz="0 0 ${finger_length/2}" rpy="0 0 0"/>
-      <geometry><box size="0.015 0.008 ${finger_length}"/></geometry>
-    </collision>
-    <xacro:box_inertia m="${finger_mass}" l="0.015" w="0.008" h="${finger_length}"/>
+    <visual><origin xyz="0.02 -0.015 0"/>
+      <geometry><box size="0.04 0.01 0.02"/></geometry>
+      <material name="silver"/></visual>
+    <collision><origin xyz="0.02 -0.015 0"/>
+      <geometry><box size="0.04 0.01 0.02"/></geometry></collision>
+    <xacro:box_inertia m="0.05" l="0.04" w="0.01" h="0.02"/>
   </link>
   <joint name="right_finger_joint" type="prismatic">
-    <parent link="end_effector_link"/>
-    <child  link="right_finger_link"/>
-    <origin xyz="0 -0.02 0" rpy="0 0 0"/>
-    <axis xyz="0 -1 0"/>
-    <limit lower="0.0" upper="0.04" effort="5" velocity="0.1"/>
-  </joint>
-  <!-- ================================================================ -->
-  <!--  RGB-D CAMERA                                                     -->
-  <!-- ================================================================ -->
+    <parent link="gripper_link"/><child link="right_finger_link"/>
+    <origin xyz="0.03 -0.012 0" rpy="0 0 0"/><axis xyz="0 -1 0"/>
+    <limit lower="0.0" upper="0.03" effort="10" velocity="0.5"/>
+  </joint>
+  <!-- LIDAR -->
+  <link name="lidar_link">
+    <visual><geometry><cylinder radius="0.04" length="0.04"/></geometry>
+      <material name="black3"><color rgba="0.05 0.05 0.05 1"/></material></visual>
+    <collision><geometry><cylinder radius="0.04" length="0.04"/></geometry></collision>
+    <xacro:cylinder_inertia m="0.2" r="0.04" h="0.04"/>
+  </link>
+  <joint name="lidar_joint" type="fixed">
+    <parent link="base_link"/><child link="lidar_link"/>
+    <origin xyz="0.18 0 0.22" rpy="0 0 0"/>
+  </joint>
+  <!-- CAMERA -->
   <link name="camera_link">
-    <visual>
-      <geometry><box size="0.04 0.10 0.03"/></geometry>
-      <material name="black"/>
-    </visual>
-    <inertial>
-      <mass value="${camera_mass}"/>
-      <inertia ixx="1e-4" ixy="0" ixz="0" iyy="1e-4" iyz="0" izz="1e-4"/>
-    </inertial>
+    <visual><geometry><box size="0.05 0.03 0.03"/></geometry>
+      <material name="orange"><color rgba="0.9 0.5 0.2 1.0"/></material></visual>
+    <collision><geometry><box size="0.05 0.03 0.03"/></geometry></collision>
+    <xacro:box_inertia m="0.1" l="0.05" w="0.03" h="0.03"/>
   </link>
   <joint name="camera_joint" type="fixed">
-    <parent link="link4"/>
-    <child  link="camera_link"/>
-    <origin xyz="0.025 0 ${link4_length - 0.02}" rpy="0 0.3 0"/>
-  </joint>
-  <!-- Camera optical frame (Z forward convention for image pipeline) -->
+    <parent link="arm_base_link"/><child link="camera_link"/>
+    <origin xyz="0.15 0 0.28" rpy="0 0 0"/>
+  </joint>
   <link name="camera_optical_frame"/>
   <joint name="camera_optical_joint" type="fixed">
-    <parent link="camera_link"/>
-    <child  link="camera_optical_frame"/>
+    <parent link="camera_link"/><child link="camera_optical_frame"/>
     <origin xyz="0 0 0" rpy="${-pi/2} 0 ${-pi/2}"/>
   </joint>
-  <!-- Gazebo RGB-D plugin -->
+  <!-- ==================== GAZEBO PLUGINS ==================== -->
+  <!-- Differential Drive -->
+  <gazebo>
+    <plugin name="diff_drive" filename="libgazebo_ros_diff_drive.so">
+      <ros>
+        <remapping>cmd_vel:=/cmd_vel</remapping>
+        <remapping>odom:=/odom</remapping>
+      </ros>
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