Commit message: fix(urdf): correct wheel_separation, base inertia origin, spawn stability

File: ros2_mobile_manipulator_ws/src/simulation_pkg/urdf/mobile_manipulator.urdf.xacro (robot description, xacro)
@@ -9,10 +9,13 @@
   <xacro:property name="wheel_width"  value="0.03"/>
   <xacro:property name="wheel_mass"   value="0.5"/>
+  <!-- Actual lateral distance between wheel centres (y offset × 2) -->
+  <xacro:property name="wheel_sep"    value="0.42"/>
   <xacro:property name="arm_link1" value="0.28"/>
   <xacro:property name="arm_link2" value="0.24"/>
   <xacro:property name="arm_link3" value="0.14"/>
   <!-- INERTIA MACROS -->
-  <xacro:macro name="box_inertia" params="m l w h">
+  <xacro:macro name="box_inertia" params="m l w h ox:=0 oy:=0 oz:=0">
     <inertial>
+      <origin xyz="${ox} ${oy} ${oz}"/>
       <mass value="${m}"/>
       <inertia ixx="${m*(w*w+h*h)/12}" ixy="0" ixz="0"
@@ -67,5 +70,8 @@
       <geometry><box size="${base_length} ${base_width} ${base_height}"/></geometry>
     </collision>
-    <xacro:box_inertia m="${base_mass}" l="${base_length}" w="${base_width}" h="${base_height}"/>
+    <!-- origin aligned with centre-of-mass (middle of box height) -->
+    <xacro:box_inertia m="${base_mass}"
+                       l="${base_length}" w="${base_width}" h="${base_height}"
+                       oz="${base_height/2}"/>
   </link>
   <!-- WHEELS -->
@@ -74,37 +80,25 @@
   <xacro:wheel name="wheel_rear_left"   x="-0.16" y="0.21"/>
   <xacro:wheel name="wheel_rear_right"  x="-0.16" y="-0.21"/>
-  <!-- Rear wheels act as passive casters (low friction so they don't resist motion) -->
+  <!-- Rear wheels: passive casters (very low friction) -->
   <gazebo reference="wheel_rear_left_link">
-    <mu1>0.01</mu1>
-    <mu2>0.01</mu2>
-    <kp>500000.0</kp>
-    <kd>10.0</kd>
-    <minDepth>0.001</minDepth>
-    <maxVel>0.1</maxVel>
+    <mu1>0.01</mu1><mu2>0.01</mu2>
+    <kp>500000.0</kp><kd>10.0</kd>
+    <minDepth>0.001</minDepth><maxVel>0.1</maxVel>
   </gazebo>
   <gazebo reference="wheel_rear_right_link">
-    <mu1>0.01</mu1>
-    <mu2>0.01</mu2>
-    <kp>500000.0</kp>
-    <kd>10.0</kd>
-    <minDepth>0.001</minDepth>
-    <maxVel>0.1</maxVel>
-  </gazebo>
-  <!-- Front wheels have good traction -->
+    <mu1>0.01</mu1><mu2>0.01</mu2>
+    <kp>500000.0</kp><kd>10.0</kd>
+    <minDepth>0.001</minDepth><maxVel>0.1</maxVel>
+  </gazebo>
+  <!-- Front wheels: driven (good traction) -->
   <gazebo reference="wheel_front_left_link">
-    <mu1>1.0</mu1>
-    <mu2>1.0</mu2>
-    <kp>500000.0</kp>
-    <kd>10.0</kd>
-    <minDepth>0.001</minDepth>
-    <maxVel>0.1</maxVel>
+    <mu1>1.5</mu1><mu2>1.5</mu2>
+    <kp>500000.0</kp><kd>10.0</kd>
+    <minDepth>0.001</minDepth><maxVel>0.1</maxVel>
   </gazebo>
   <gazebo reference="wheel_front_right_link">
-    <mu1>1.0</mu1>
-    <mu2>1.0</mu2>
-    <kp>500000.0</kp>
-    <kd>10.0</kd>
-    <minDepth>0.001</minDepth>
-    <maxVel>0.1</maxVel>
+    <mu1>1.5</mu1><mu2>1.5</mu2>
+    <kp>500000.0</kp><kd>10.0</kd>
+    <minDepth>0.001</minDepth><maxVel>0.1</maxVel>
   </gazebo>
   <!-- ARM BASE -->
@@ -145,5 +139,5 @@
     <collision><origin xyz="${arm_link2/2} 0 0"/>
       <geometry><box size="${arm_link2} 0.05 0.05"/></geometry></collision>
-    <xacro:box_inertia m="0.4" l="${arm_link2}" w="0.05" h="0.05"/>
+    <xacro:box_inertia m="0.4" l="${arm_link2}" w="0.05" h="0.05" ox="${arm_link2/2}"/>
   </link>
   <joint name="arm_joint_2" type="revolute">
@@ -159,5 +153,5 @@
     <collision><origin xyz="${arm_link3/2} 0 0"/>
       <geometry><box size="${arm_link3} 0.045 0.045"/></geometry></collision>
-    <xacro:box_inertia m="0.3" l="${arm_link3}" w="0.045" h="0.045"/>
+    <xacro:box_inertia m="0.3" l="${arm_link3}" w="0.045" h="0.045" ox="${arm_link3/2}"/>
   </link>
   <joint name="arm_joint_3" type="revolute">
@@ -173,5 +167,5 @@
     <collision><origin xyz="${arm_link3} 0 0"/>
       <geometry><box size="${arm_link3} 0.035 0.035"/></geometry></collision>
-    <xacro:box_inertia m="0.2" l="${arm_link3}" w="0.035" h="0.035"/>
+    <xacro:box_inertia m="0.2" l="${arm_link3}" w="0.035" h="0.035" ox="${arm_link3}"/>
   </link>
   <joint name="arm_joint_4" type="revolute">
@@ -198,5 +192,5 @@
     <collision><origin xyz="0.02 0.015 0"/>
       <geometry><box size="0.04 0.01 0.02"/></geometry></collision>
-    <xacro:box_inertia m="0.05" l="0.04" w="0.01" h="0.02"/>
+    <xacro:box_inertia m="0.05" l="0.04" w="0.01" h="0.02" ox="0.02" oy="0.015"/>
   </link>
   <joint name="left_finger_joint" type="prismatic">
@@ -211,5 +205,5 @@
     <collision><origin xyz="0.02 -0.015 0"/>
       <geometry><box size="0.04 0.01 0.02"/></geometry></collision>
-    <xacro:box_inertia m="0.05" l="0.04" w="0.01" h="0.02"/>
+    <xacro:box_inertia m="0.05" l="0.04" w="0.01" h="0.02" ox="0.02" oy="-0.015"/>
   </link>
   <joint name="right_finger_joint" type="prismatic">
@@ -247,6 +241,7 @@
   <!-- ==================== GAZEBO PLUGINS ==================== -->
   <!-- Differential Drive
-       Controls the two FRONT wheels.
-       Rear wheels are passive (low friction) so they follow freely.
+       - Controls front two wheels only.
+       - Rear wheels are passive (low friction) and follow freely.
+       - wheel_separation: actual centre-to-centre lateral distance = 0.42 m
   -->
   <gazebo>
@@ -259,5 +254,5 @@
       <left_joint>wheel_front_left_joint</left_joint>
       <right_joint>wheel_front_right_joint</right_joint>
-      <wheel_separation>0.42</wheel_separation>
+      <wheel_separation>${wheel_sep}</wheel_separation>
       <wheel_diameter>${2*wheel_radius}</wheel_diameter>
       <max_wheel_torque>20</max_wheel_torque>

Commit message: fix(simulation): correct spawn height + inertia origins to stop robot flying in Gazebo

File: ros2_mobile_manipulator_ws/src/simulation_pkg/urdf/mobile_manipulator.urdf.xacro (robot description, xacro)
@@ -1,5 +1,7 @@
 <?xml version="1.0"?>
 <robot xmlns:xacro="http://www.ros.org/wiki/xacro" name="mobile_manipulator">
-  <!-- PROPERTIES -->
+  <!-- ============================================================
+       PROPERTIES
+  ============================================================ -->
   <xacro:property name="base_length" value="0.46"/>
   <xacro:property name="base_width"  value="0.38"/>
@@ -9,10 +11,13 @@
   <xacro:property name="wheel_width"  value="0.03"/>
   <xacro:property name="wheel_mass"   value="0.5"/>
-  <!-- Actual lateral distance between wheel centres (y offset × 2) -->
+  <!-- centre-to-centre lateral distance between left and right wheels -->
   <xacro:property name="wheel_sep"    value="0.42"/>
   <xacro:property name="arm_link1" value="0.28"/>
   <xacro:property name="arm_link2" value="0.24"/>
   <xacro:property name="arm_link3" value="0.14"/>
-  <!-- INERTIA MACROS -->
+  <!-- ============================================================
+       INERTIA MACROS
+       ox/oy/oz = centre-of-mass offset from the link origin
+  ============================================================ -->
   <xacro:macro name="box_inertia" params="m l w h ox:=0 oy:=0 oz:=0">
     <inertial>
@@ -24,6 +29,7 @@
     </inertial>
   </xacro:macro>
-  <xacro:macro name="cylinder_inertia" params="m r h">
+  <xacro:macro name="cylinder_inertia" params="m r h oz:=0">
     <inertial>
+      <origin xyz="0 0 ${oz}"/>
       <mass value="${m}"/>
       <inertia ixx="${m*(3*r*r+h*h)/12}" ixy="0" ixz="0"
@@ -32,5 +38,7 @@
     </inertial>
   </xacro:macro>
-  <!-- WHEEL MACRO -->
+  <!-- ============================================================
+       WHEEL MACRO
+  ============================================================ -->
   <xacro:macro name="wheel" params="name x y">
     <link name="${name}_link">
@@ -42,4 +50,5 @@
         <geometry><cylinder radius="${wheel_radius}" length="${wheel_width}"/></geometry>
       </collision>
+      <!-- cylinder along Z after rpy pi/2 rotation → inertia is symmetric, oz=0 -->
       <xacro:cylinder_inertia m="${wheel_mass}" r="${wheel_radius}" h="${wheel_width}"/>
     </link>
@@ -52,12 +61,20 @@
     </joint>
   </xacro:macro>
-  <!-- BASE FOOTPRINT -->
+  <!-- ============================================================
+       BASE FOOTPRINT  (sits on the ground plane)
+  ============================================================ -->
   <link name="base_footprint"/>
   <joint name="base_footprint_joint" type="fixed">
     <parent link="base_footprint"/>
     <child  link="base_link"/>
+    <!-- base_link origin is at wheel-axle height = wheel_radius above footprint -->
     <origin xyz="0 0 ${wheel_radius}" rpy="0 0 0"/>
   </joint>
-  <!-- BASE LINK -->
+  <!-- ============================================================
+       BASE LINK
+       Visual/collision box is offset +z by half its height so its
+       bottom face sits at z=0 (wheel-axle plane).
+       Inertia origin must match that same offset.
+  ============================================================ -->
   <link name="base_link">
     <visual>
@@ -70,37 +87,40 @@
       <geometry><box size="${base_length} ${base_width} ${base_height}"/></geometry>
     </collision>
-    <!-- origin aligned with centre-of-mass (middle of box height) -->
     <xacro:box_inertia m="${base_mass}"
                        l="${base_length}" w="${base_width}" h="${base_height}"
                        oz="${base_height/2}"/>
   </link>
-  <!-- WHEELS -->
+  <!-- ============================================================
+       WHEELS  (4 × macro)
+  ============================================================ -->
   <xacro:wheel name="wheel_front_left"  x="0.16"  y="0.21"/>
   <xacro:wheel name="wheel_front_right" x="0.16"  y="-0.21"/>
   <xacro:wheel name="wheel_rear_left"   x="-0.16" y="0.21"/>
   <xacro:wheel name="wheel_rear_right"  x="-0.16" y="-0.21"/>
-  <!-- Rear wheels: passive casters (very low friction) -->
+  <!-- Rear wheels: passive casters → very low friction -->
   <gazebo reference="wheel_rear_left_link">
     <mu1>0.01</mu1><mu2>0.01</mu2>
-    <kp>500000.0</kp><kd>10.0</kd>
-    <minDepth>0.001</minDepth><maxVel>0.1</maxVel>
+    <kp>1000000.0</kp><kd>100.0</kd>
+    <minDepth>0.001</minDepth><maxVel>1.0</maxVel>
   </gazebo>
   <gazebo reference="wheel_rear_right_link">
     <mu1>0.01</mu1><mu2>0.01</mu2>
-    <kp>500000.0</kp><kd>10.0</kd>
-    <minDepth>0.001</minDepth><maxVel>0.1</maxVel>
-  </gazebo>
-  <!-- Front wheels: driven (good traction) -->
+    <kp>1000000.0</kp><kd>100.0</kd>
+    <minDepth>0.001</minDepth><maxVel>1.0</maxVel>
+  </gazebo>
+  <!-- Front wheels: driven → good traction -->
   <gazebo reference="wheel_front_left_link">
     <mu1>1.5</mu1><mu2>1.5</mu2>
-    <kp>500000.0</kp><kd>10.0</kd>
-    <minDepth>0.001</minDepth><maxVel>0.1</maxVel>
+    <kp>1000000.0</kp><kd>100.0</kd>
+    <minDepth>0.001</minDepth><maxVel>1.0</maxVel>
   </gazebo>
   <gazebo reference="wheel_front_right_link">
     <mu1>1.5</mu1><mu2>1.5</mu2>
-    <kp>500000.0</kp><kd>10.0</kd>
-    <minDepth>0.001</minDepth><maxVel>0.1</maxVel>
-  </gazebo>
-  <!-- ARM BASE -->
+    <kp>1000000.0</kp><kd>100.0</kd>
+    <minDepth>0.001</minDepth><maxVel>1.0</maxVel>
+  </gazebo>
+  <!-- ============================================================
+       ARM BASE
+  ============================================================ -->
   <link name="arm_base_link">
     <visual>
@@ -113,5 +133,5 @@
       <geometry><cylinder length="0.1" radius="0.08"/></geometry>
     </collision>
-    <xacro:cylinder_inertia m="1.0" r="0.08" h="0.1"/>
+    <xacro:cylinder_inertia m="1.0" r="0.08" h="0.1" oz="0.05"/>
   </link>
   <joint name="arm_base_joint" type="fixed">
@@ -120,60 +140,98 @@
     <origin xyz="0 0 0.18" rpy="0 0 0"/>
   </joint>
-  <!-- ARM LINKS -->
+  <!-- ============================================================
+       ARM LINK 1  (vertical cylinder, rotates about Z)
+  ============================================================ -->
   <link name="arm_link_1">
-    <visual><geometry><cylinder length="${arm_link1}" radius="0.04"/></geometry>
-      <material name="red"><color rgba="0.8 0.2 0.2 1.0"/></material></visual>
-    <collision><geometry><cylinder length="${arm_link1}" radius="0.04"/></geometry></collision>
-    <xacro:cylinder_inertia m="0.5" r="0.04" h="${arm_link1}"/>
+    <visual>
+      <origin xyz="0 0 ${arm_link1/2}"/>
+      <geometry><cylinder length="${arm_link1}" radius="0.04"/></geometry>
+      <material name="red"><color rgba="0.8 0.2 0.2 1.0"/></material>
+    </visual>
+    <collision>
+      <origin xyz="0 0 ${arm_link1/2}"/>
+      <geometry><cylinder length="${arm_link1}" radius="0.04"/></geometry>
+    </collision>
+    <xacro:cylinder_inertia m="0.5" r="0.04" h="${arm_link1}" oz="${arm_link1/2}"/>
   </link>
   <joint name="arm_joint_1" type="revolute">
     <parent link="arm_base_link"/><child link="arm_link_1"/>
-    <origin xyz="0 0 0.1" rpy="0 0 0"/><axis xyz="0 0 1"/>
+    <origin xyz="0 0 0.1" rpy="0 0 0"/>
+    <axis xyz="0 0 1"/>
     <limit lower="${-pi}" upper="${pi}" effort="30" velocity="1.5"/>
     <dynamics damping="0.1" friction="0.05"/>
   </joint>
+  <!-- ============================================================
+       ARM LINK 2
+  ============================================================ -->
   <link name="arm_link_2">
-    <visual><origin xyz="${arm_link2/2} 0 0"/>
+    <visual>
+      <origin xyz="${arm_link2/2} 0 0"/>
       <geometry><box size="${arm_link2} 0.05 0.05"/></geometry>
-      <material name="green"><color rgba="0.2 0.8 0.3 1.0"/></material></visual>
-    <collision><origin xyz="${arm_link2/2} 0 0"/>
-      <geometry><box size="${arm_link2} 0.05 0.05"/></geometry></collision>
-    <xacro:box_inertia m="0.4" l="${arm_link2}" w="0.05" h="0.05" ox="${arm_link2/2}"/>
+      <material name="green"><color rgba="0.2 0.8 0.3 1.0"/></material>
+    </visual>
+    <collision>
+      <origin xyz="${arm_link2/2} 0 0"/>
+      <geometry><box size="${arm_link2} 0.05 0.05"/></geometry>
+    </collision>
+    <xacro:box_inertia m="0.4" l="${arm_link2}" w="0.05" h="0.05"
+                       ox="${arm_link2/2}"/>
   </link>
   <joint name="arm_joint_2" type="revolute">
     <parent link="arm_link_1"/><child link="arm_link_2"/>
-    <origin xyz="0 0 ${arm_link1}" rpy="0 0 0"/><axis xyz="0 1 0"/>
+    <origin xyz="0 0 ${arm_link1}" rpy="0 0 0"/>
+    <axis xyz="0 1 0"/>
     <limit lower="${-pi/2}" upper="${pi/2}" effort="25" velocity="1.5"/>
     <dynamics damping="0.1" friction="0.05"/>
   </joint>
+  <!-- ============================================================
+       ARM LINK 3
+  ============================================================ -->
   <link name="arm_link_3">
-    <visual><origin xyz="${arm_link3/2} 0 0"/>
+    <visual>
+      <origin xyz="${arm_link3/2} 0 0"/>
       <geometry><box size="${arm_link3} 0.045 0.045"/></geometry>
-      <material name="yellow"><color rgba="0.9 0.8 0.2 1.0"/></material></visual>
-    <collision><origin xyz="${arm_link3/2} 0 0"/>
-      <geometry><box size="${arm_link3} 0.045 0.045"/></geometry></collision>
-    <xacro:box_inertia m="0.3" l="${arm_link3}" w="0.045" h="0.045" ox="${arm_link3/2}"/>
+      <material name="yellow"><color rgba="0.9 0.8 0.2 1.0"/></material>
+    </visual>
+    <collision>
+      <origin xyz="${arm_link3/2} 0 0"/>
+      <geometry><box size="${arm_link3} 0.045 0.045"/></geometry>
+    </collision>
+    <xacro:box_inertia m="0.3" l="${arm_link3}" w="0.045" h="0.045"
+                       ox="${arm_link3/2}"/>
   </link>
   <joint name="arm_joint_3" type="revolute">
     <parent link="arm_link_2"/><child link="arm_link_3"/>
-    <origin xyz="${arm_link2} 0 0" rpy="0 0 0"/><axis xyz="0 1 0"/>
+    <origin xyz="${arm_link2} 0 0" rpy="0 0 0"/>
+    <axis xyz="0 1 0"/>
     <limit lower="${-pi/2}" upper="${pi/2}" effort="20" velocity="1.5"/>
     <dynamics damping="0.1" friction="0.05"/>
   </joint>
+  <!-- ============================================================
+       ARM LINK 4
+  ============================================================ -->
   <link name="arm_link_4">
-    <visual><origin xyz="${arm_link3} 0 0"/>
+    <visual>
+      <origin xyz="${arm_link3/2} 0 0"/>
       <geometry><box size="${arm_link3} 0.035 0.035"/></geometry>
-      <material name="purple"><color rgba="0.7 0.2 0.8 1.0"/></material></visual>
-    <collision><origin xyz="${arm_link3} 0 0"/>
-      <geometry><box size="${arm_link3} 0.035 0.035"/></geometry></collision>
-    <xacro:box_inertia m="0.2" l="${arm_link3}" w="0.035" h="0.035" ox="${arm_link3}"/>
+      <material name="purple"><color rgba="0.7 0.2 0.8 1.0"/></material>
+    </visual>
+    <collision>
+      <origin xyz="${arm_link3/2} 0 0"/>
+      <geometry><box size="${arm_link3} 0.035 0.035"/></geometry>
+    </collision>
+    <xacro:box_inertia m="0.2" l="${arm_link3}" w="0.035" h="0.035"
+                       ox="${arm_link3/2}"/>
   </link>
   <joint name="arm_joint_4" type="revolute">
     <parent link="arm_link_3"/><child link="arm_link_4"/>
-    <origin xyz="${arm_link3} 0 0" rpy="0 0 0"/><axis xyz="0 1 0"/>
+    <origin xyz="${arm_link3} 0 0" rpy="0 0 0"/>
+    <axis xyz="0 1 0"/>
     <limit lower="${-pi}" upper="${pi}" effort="15" velocity="2.0"/>
     <dynamics damping="0.05" friction="0.02"/>
   </joint>
-  <!-- GRIPPER -->
+  <!-- ============================================================
+       GRIPPER
+  ============================================================ -->
   <link name="gripper_link">
     <visual><geometry><box size="0.06 0.02 0.02"/></geometry>
@@ -192,5 +250,6 @@
     <collision><origin xyz="0.02 0.015 0"/>
       <geometry><box size="0.04 0.01 0.02"/></geometry></collision>
-    <xacro:box_inertia m="0.05" l="0.04" w="0.01" h="0.02" ox="0.02" oy="0.015"/>
+    <xacro:box_inertia m="0.05" l="0.04" w="0.01" h="0.02"
+                       ox="0.02" oy="0.015"/>
   </link>
   <joint name="left_finger_joint" type="prismatic">
@@ -205,5 +264,6 @@
     <collision><origin xyz="0.02 -0.015 0"/>
       <geometry><box size="0.04 0.01 0.02"/></geometry></collision>
-    <xacro:box_inertia m="0.05" l="0.04" w="0.01" h="0.02" ox="0.02" oy="-0.015"/>
+    <xacro:box_inertia m="0.05" l="0.04" w="0.01" h="0.02"
+                       ox="0.02" oy="-0.015"/>
   </link>
   <joint name="right_finger_joint" type="prismatic">
@@ -212,5 +272,7 @@
     <limit lower="0.0" upper="0.03" effort="10" velocity="0.5"/>
   </joint>
-  <!-- LIDAR -->
+  <!-- ============================================================
+       LIDAR
+  ============================================================ -->
   <link name="lidar_link">
     <visual><geometry><cylinder radius="0.04" length="0.04"/></geometry>
@@ -223,5 +285,7 @@
     <origin xyz="0.18 0 0.22" rpy="0 0 0"/>
   </joint>
-  <!-- CAMERA -->
+  <!-- ============================================================
+       CAMERA
+  ============================================================ -->
   <link name="camera_link">
     <visual><geometry><box size="0.05 0.03 0.03"/></geometry>
@@ -239,9 +303,12 @@
     <origin xyz="0 0 0" rpy="${-pi/2} 0 ${-pi/2}"/>
   </joint>
-  <!-- ==================== GAZEBO PLUGINS ==================== -->
-  <!-- Differential Drive
-       - Controls front two wheels only.
-       - Rear wheels are passive (low friction) and follow freely.
-       - wheel_separation: actual centre-to-centre lateral distance = 0.42 m
+  <!-- ============================================================
+       GAZEBO PLUGINS
+  ============================================================ -->
+  <!--
+    Differential Drive
+    - Only front wheels are driven.
+    - Rear wheels are passive (mu≈0) and follow freely.
+    - wheel_separation = lateral distance between wheel centres = 0.42 m
   -->
   <gazebo>
