Commit message: robot urdf

File: ros2_mobile_manipulator_ws/src/simulation_pkg/urdf/mobile_manipulator.urdf.xacro (robot description, xacro)
@@ -1,393 +1,789 @@
-<?xml version="1.0"?>
-<robot xmlns:xacro="http://www.ros.org/wiki/xacro" name="mobile_manipulator">
-  <!-- ============================================================
-       PROPERTIES
-  ============================================================ -->
-  <xacro:property name="base_length" value="0.46"/>
-  <xacro:property name="base_width"  value="0.38"/>
-  <xacro:property name="base_height" value="0.12"/>
-  <xacro:property name="base_mass"   value="18.0"/>
-  <xacro:property name="wheel_radius" value="0.05"/>
-  <xacro:property name="wheel_width"  value="0.03"/>
-  <xacro:property name="wheel_mass"   value="0.5"/>
-  <!-- centre-to-centre lateral distance between left and right wheels -->
-  <xacro:property name="wheel_sep"    value="0.42"/>
-  <xacro:property name="arm_link1" value="0.28"/>
-  <xacro:property name="arm_link2" value="0.24"/>
-  <xacro:property name="arm_link3" value="0.14"/>
-  <!-- ============================================================
-       INERTIA MACROS
-       ox/oy/oz = centre-of-mass offset from the link origin
-  ============================================================ -->
-  <xacro:macro name="box_inertia" params="m l w h ox:=0 oy:=0 oz:=0">
-    <inertial>
-      <origin xyz="${ox} ${oy} ${oz}"/>
-      <mass value="${m}"/>
-      <inertia ixx="${m*(w*w+h*h)/12}" ixy="0" ixz="0"
-               iyy="${m*(l*l+h*h)/12}" iyz="0"
-               izz="${m*(l*l+w*w)/12}"/>
-    </inertial>
-  </xacro:macro>
-  <xacro:macro name="cylinder_inertia" params="m r h oz:=0">
-    <inertial>
-      <origin xyz="0 0 ${oz}"/>
-      <mass value="${m}"/>
-      <inertia ixx="${m*(3*r*r+h*h)/12}" ixy="0" ixz="0"
-               iyy="${m*(3*r*r+h*h)/12}" iyz="0"
-               izz="${m*r*r/2}"/>
-    </inertial>
-  </xacro:macro>
-  <!-- ============================================================
-       WHEEL MACRO
-  ============================================================ -->
-  <xacro:macro name="wheel" params="name x y">
-    <link name="${name}_link">
-      <visual>
-        <geometry><cylinder radius="${wheel_radius}" length="${wheel_width}"/></geometry>
-        <material name="black"><color rgba="0.05 0.05 0.05 1"/></material>
-      </visual>
-      <collision>
-        <geometry><cylinder radius="${wheel_radius}" length="${wheel_width}"/></geometry>
-      </collision>
-      <!-- cylinder along Z after rpy pi/2 rotation → inertia is symmetric, oz=0 -->
-      <xacro:cylinder_inertia m="${wheel_mass}" r="${wheel_radius}" h="${wheel_width}"/>
-    </link>
-    <joint name="${name}_joint" type="continuous">
-      <parent link="base_link"/>
-      <child  link="${name}_link"/>
-      <origin xyz="${x} ${y} 0" rpy="${pi/2} 0 0"/>
-      <axis xyz="0 0 1"/>
-      <dynamics damping="0.01" friction="0.1"/>
-    </joint>
-  </xacro:macro>
-  <!-- ============================================================
-       BASE FOOTPRINT  (sits on the ground plane)
-  ============================================================ -->
-  <link name="base_footprint"/>
-  <joint name="base_footprint_joint" type="fixed">
-    <parent link="base_footprint"/>
-    <child  link="base_link"/>
-    <!-- base_link origin is at wheel-axle height = wheel_radius above footprint -->
-    <origin xyz="0 0 ${wheel_radius}" rpy="0 0 0"/>
-  </joint>
-  <!-- ============================================================
-       BASE LINK
-       Visual/collision box is offset +z by half its height so its
-       bottom face sits at z=0 (wheel-axle plane).
-       Inertia origin must match that same offset.
-  ============================================================ -->
-  <link name="base_link">
-    <visual>
-      <origin xyz="0 0 ${base_height/2}"/>
-      <geometry><box size="${base_length} ${base_width} ${base_height}"/></geometry>
-      <material name="gray"><color rgba="0.6 0.6 0.65 1.0"/></material>
-    </visual>
-    <collision>
-      <origin xyz="0 0 ${base_height/2}"/>
-      <geometry><box size="${base_length} ${base_width} ${base_height}"/></geometry>
-    </collision>
-    <xacro:box_inertia m="${base_mass}"
-                       l="${base_length}" w="${base_width}" h="${base_height}"
-                       oz="${base_height/2}"/>
-  </link>
-  <!-- ============================================================
-       WHEELS  (4 × macro)
-  ============================================================ -->
-  <xacro:wheel name="wheel_front_left"  x="0.16"  y="0.21"/>
-  <xacro:wheel name="wheel_front_right" x="0.16"  y="-0.21"/>
-  <xacro:wheel name="wheel_rear_left"   x="-0.16" y="0.21"/>
-  <xacro:wheel name="wheel_rear_right"  x="-0.16" y="-0.21"/>
-  <!-- Rear wheels: passive casters → very low friction -->
-  <gazebo reference="wheel_rear_left_link">
-    <mu1>0.01</mu1><mu2>0.01</mu2>
-    <kp>1000000.0</kp><kd>100.0</kd>
-    <minDepth>0.001</minDepth><maxVel>1.0</maxVel>
-  </gazebo>
-  <gazebo reference="wheel_rear_right_link">
-    <mu1>0.01</mu1><mu2>0.01</mu2>
-    <kp>1000000.0</kp><kd>100.0</kd>
-    <minDepth>0.001</minDepth><maxVel>1.0</maxVel>
-  </gazebo>
-  <!-- Front wheels: driven → good traction -->
-  <gazebo reference="wheel_front_left_link">
-    <mu1>1.5</mu1><mu2>1.5</mu2>
-    <kp>1000000.0</kp><kd>100.0</kd>
-    <minDepth>0.001</minDepth><maxVel>1.0</maxVel>
-  </gazebo>
-  <gazebo reference="wheel_front_right_link">
-    <mu1>1.5</mu1><mu2>1.5</mu2>
-    <kp>1000000.0</kp><kd>100.0</kd>
-    <minDepth>0.001</minDepth><maxVel>1.0</maxVel>
-  </gazebo>
-  <!-- ============================================================
-       ARM BASE
-  ============================================================ -->
-  <link name="arm_base_link">
-    <visual>
-      <origin xyz="0 0 0.05"/>
-      <geometry><cylinder length="0.1" radius="0.08"/></geometry>
-      <material name="blue"><color rgba="0.2 0.4 0.8 1.0"/></material>
-    </visual>
-    <collision>
-      <origin xyz="0 0 0.05"/>
-      <geometry><cylinder length="0.1" radius="0.08"/></geometry>
-    </collision>
-    <xacro:cylinder_inertia m="1.0" r="0.08" h="0.1" oz="0.05"/>
-  </link>
-  <joint name="arm_base_joint" type="fixed">
-    <parent link="base_link"/>
-    <child  link="arm_base_link"/>
-    <origin xyz="0 0 0.18" rpy="0 0 0"/>
-  </joint>
-  <!-- ============================================================
-       ARM LINK 1  (vertical cylinder, rotates about Z)
-  ============================================================ -->
-  <link name="arm_link_1">
-    <visual>
-      <origin xyz="0 0 ${arm_link1/2}"/>
-      <geometry><cylinder length="${arm_link1}" radius="0.04"/></geometry>
-      <material name="red"><color rgba="0.8 0.2 0.2 1.0"/></material>
-    </visual>
-    <collision>
-      <origin xyz="0 0 ${arm_link1/2}"/>
-      <geometry><cylinder length="${arm_link1}" radius="0.04"/></geometry>
-    </collision>
-    <xacro:cylinder_inertia m="0.5" r="0.04" h="${arm_link1}" oz="${arm_link1/2}"/>
-  </link>
-  <joint name="arm_joint_1" type="revolute">
-    <parent link="arm_base_link"/><child link="arm_link_1"/>
-    <origin xyz="0 0 0.1" rpy="0 0 0"/>
-    <axis xyz="0 0 1"/>
-    <limit lower="${-pi}" upper="${pi}" effort="30" velocity="1.5"/>
-    <dynamics damping="0.1" friction="0.05"/>
-  </joint>
-  <!-- ============================================================
-       ARM LINK 2
-  ============================================================ -->
-  <link name="arm_link_2">
-    <visual>
-      <origin xyz="${arm_link2/2} 0 0"/>
-      <geometry><box size="${arm_link2} 0.05 0.05"/></geometry>
-      <material name="green"><color rgba="0.2 0.8 0.3 1.0"/></material>
-    </visual>
-    <collision>
-      <origin xyz="${arm_link2/2} 0 0"/>
-      <geometry><box size="${arm_link2} 0.05 0.05"/></geometry>
-    </collision>
-    <xacro:box_inertia m="0.4" l="${arm_link2}" w="0.05" h="0.05"
-                       ox="${arm_link2/2}"/>
-  </link>
-  <joint name="arm_joint_2" type="revolute">
-    <parent link="arm_link_1"/><child link="arm_link_2"/>
-    <origin xyz="0 0 ${arm_link1}" rpy="0 0 0"/>
-    <axis xyz="0 1 0"/>
-    <limit lower="${-pi/2}" upper="${pi/2}" effort="25" velocity="1.5"/>
-    <dynamics damping="0.1" friction="0.05"/>
-  </joint>
-  <!-- ============================================================
-       ARM LINK 3
-  ============================================================ -->
-  <link name="arm_link_3">
-    <visual>
-      <origin xyz="${arm_link3/2} 0 0"/>
-      <geometry><box size="${arm_link3} 0.045 0.045"/></geometry>
-      <material name="yellow"><color rgba="0.9 0.8 0.2 1.0"/></material>
-    </visual>
-    <collision>
-      <origin xyz="${arm_link3/2} 0 0"/>
-      <geometry><box size="${arm_link3} 0.045 0.045"/></geometry>
-    </collision>
-    <xacro:box_inertia m="0.3" l="${arm_link3}" w="0.045" h="0.045"
-                       ox="${arm_link3/2}"/>
-  </link>
-  <joint name="arm_joint_3" type="revolute">
-    <parent link="arm_link_2"/><child link="arm_link_3"/>
-    <origin xyz="${arm_link2} 0 0" rpy="0 0 0"/>
-    <axis xyz="0 1 0"/>
-    <limit lower="${-pi/2}" upper="${pi/2}" effort="20" velocity="1.5"/>
-    <dynamics damping="0.1" friction="0.05"/>
-  </joint>
-  <!-- ============================================================
-       ARM LINK 4
-  ============================================================ -->
-  <link name="arm_link_4">
-    <visual>
-      <origin xyz="${arm_link3/2} 0 0"/>
-      <geometry><box size="${arm_link3} 0.035 0.035"/></geometry>
-      <material name="purple"><color rgba="0.7 0.2 0.8 1.0"/></material>
-    </visual>
-    <collision>
-      <origin xyz="${arm_link3/2} 0 0"/>
-      <geometry><box size="${arm_link3} 0.035 0.035"/></geometry>
-    </collision>
-    <xacro:box_inertia m="0.2" l="${arm_link3}" w="0.035" h="0.035"
-                       ox="${arm_link3/2}"/>
-  </link>
-  <joint name="arm_joint_4" type="revolute">
-    <parent link="arm_link_3"/><child link="arm_link_4"/>
-    <origin xyz="${arm_link3} 0 0" rpy="0 0 0"/>
-    <axis xyz="0 1 0"/>
-    <limit lower="${-pi}" upper="${pi}" effort="15" velocity="2.0"/>
-    <dynamics damping="0.05" friction="0.02"/>
-  </joint>
-  <!-- ============================================================
-       GRIPPER
-  ============================================================ -->
-  <link name="gripper_link">
-    <visual><geometry><box size="0.06 0.02 0.02"/></geometry>
-      <material name="black2"><color rgba="0.1 0.1 0.1 1.0"/></material></visual>
-    <collision><geometry><box size="0.06 0.02 0.02"/></geometry></collision>
-    <xacro:box_inertia m="0.1" l="0.06" w="0.02" h="0.02"/>
-  </link>
-  <joint name="gripper_joint" type="fixed">
-    <parent link="arm_link_4"/><child link="gripper_link"/>
-    <origin xyz="${arm_link3} 0 0" rpy="0 0 0"/>
-  </joint>
-  <link name="left_finger_link">
-    <visual><origin xyz="0.02 0.015 0"/>
-      <geometry><box size="0.04 0.01 0.02"/></geometry>
-      <material name="silver"><color rgba="0.85 0.85 0.85 1.0"/></material></visual>
-    <collision><origin xyz="0.02 0.015 0"/>
-      <geometry><box size="0.04 0.01 0.02"/></geometry></collision>
-    <xacro:box_inertia m="0.05" l="0.04" w="0.01" h="0.02"
-                       ox="0.02" oy="0.015"/>
-  </link>
-  <joint name="left_finger_joint" type="prismatic">
-    <parent link="gripper_link"/><child link="left_finger_link"/>
-    <origin xyz="0.03 0.012 0" rpy="0 0 0"/><axis xyz="0 1 0"/>
-    <limit lower="0.0" upper="0.03" effort="10" velocity="0.5"/>
-  </joint>
-  <link name="right_finger_link">
-    <visual><origin xyz="0.02 -0.015 0"/>
-      <geometry><box size="0.04 0.01 0.02"/></geometry>
-      <material name="silver"/></visual>
-    <collision><origin xyz="0.02 -0.015 0"/>
-      <geometry><box size="0.04 0.01 0.02"/></geometry></collision>
-    <xacro:box_inertia m="0.05" l="0.04" w="0.01" h="0.02"
-                       ox="0.02" oy="-0.015"/>
-  </link>
-  <joint name="right_finger_joint" type="prismatic">
-    <parent link="gripper_link"/><child link="right_finger_link"/>
-    <origin xyz="0.03 -0.012 0" rpy="0 0 0"/><axis xyz="0 -1 0"/>
-    <limit lower="0.0" upper="0.03" effort="10" velocity="0.5"/>
-  </joint>
-  <!-- ============================================================
-       LIDAR
-  ============================================================ -->
-  <link name="lidar_link">
-    <visual><geometry><cylinder radius="0.04" length="0.04"/></geometry>
-      <material name="black3"><color rgba="0.05 0.05 0.05 1"/></material></visual>
-    <collision><geometry><cylinder radius="0.04" length="0.04"/></geometry></collision>
-    <xacro:cylinder_inertia m="0.2" r="0.04" h="0.04"/>
-  </link>
-  <joint name="lidar_joint" type="fixed">
-    <parent link="base_link"/><child link="lidar_link"/>
-    <origin xyz="0.18 0 0.22" rpy="0 0 0"/>
-  </joint>
-  <!-- ============================================================
-       CAMERA
-  ============================================================ -->
-  <link name="camera_link">
-    <visual><geometry><box size="0.05 0.03 0.03"/></geometry>
-      <material name="orange"><color rgba="0.9 0.5 0.2 1.0"/></material></visual>
-    <collision><geometry><box size="0.05 0.03 0.03"/></geometry></collision>
-    <xacro:box_inertia m="0.1" l="0.05" w="0.03" h="0.03"/>
-  </link>
-  <joint name="camera_joint" type="fixed">
-    <parent link="arm_base_link"/><child link="camera_link"/>
-    <origin xyz="0.15 0 0.28" rpy="0 0 0"/>
-  </joint>
-  <link name="camera_optical_frame"/>
-  <joint name="camera_optical_joint" type="fixed">
-    <parent link="camera_link"/><child link="camera_optical_frame"/>
-    <origin xyz="0 0 0" rpy="${-pi/2} 0 ${-pi/2}"/>
-  </joint>
-  <!-- ============================================================
-       GAZEBO PLUGINS
-  ============================================================ -->
-  <!--
-    Differential Drive
-    - Only front wheels are driven.
-    - Rear wheels are passive (mu≈0) and follow freely.
-    - wheel_separation = lateral distance between wheel centres = 0.42 m
-  -->
-  <gazebo>
-    <plugin name="diff_drive" filename="libgazebo_ros_diff_drive.so">
-      <ros>
-        <remapping>cmd_vel:=/cmd_vel</remapping>
-        <remapping>odom:=/odom</remapping>
-      </ros>
-      <update_rate>20</update_rate>
-      <left_joint>wheel_front_left_joint</left_joint>
-      <right_joint>wheel_front_right_joint</right_joint>
-      <wheel_separation>${wheel_sep}</wheel_separation>
-      <wheel_diameter>${2*wheel_radius}</wheel_diameter>
-      <max_wheel_torque>20</max_wheel_torque>
-      <max_wheel_acceleration>1.0</max_wheel_acceleration>
-      <command_timeout>0.5</command_timeout>
-      <publish_odom>true</publish_odom>
-      <publish_odom_tf>true</publish_odom_tf>
-      <publish_wheel_tf>true</publish_wheel_tf>
-      <odometry_frame>odom</odometry_frame>
-      <robot_base_frame>base_footprint</robot_base_frame>
-    </plugin>
-  </gazebo>
-  <!-- Joint State Publisher -->
-  <gazebo>
-    <plugin name="joint_state_publisher" filename="libgazebo_ros_joint_state_publisher.so">
-      <ros><remapping>~/out:=/joint_states</remapping></ros>
-      <joint_name>arm_joint_1</joint_name>
-      <joint_name>arm_joint_2</joint_name>
-      <joint_name>arm_joint_3</joint_name>
-      <joint_name>arm_joint_4</joint_name>
-      <joint_name>left_finger_joint</joint_name>
-      <joint_name>right_finger_joint</joint_name>
-      <joint_name>wheel_front_left_joint</joint_name>
-      <joint_name>wheel_front_right_joint</joint_name>
-      <joint_name>wheel_rear_left_joint</joint_name>
-      <joint_name>wheel_rear_right_joint</joint_name>
-      <update_rate>50</update_rate>
-    </plugin>
-  </gazebo>
-  <!-- LiDAR -->
-  <gazebo reference="lidar_link">
-    <sensor type="ray" name="lidar">
-      <visualize>false</visualize>
-      <update_rate>5.0</update_rate>
-      <ray>
-        <scan><horizontal>
-          <samples>360</samples><resolution>1</resolution>
-          <min_angle>${-pi}</min_angle><max_angle>${pi}</max_angle>
-        </horizontal></scan>
-        <range><min>0.12</min><max>12.0</max><resolution>0.01</resolution></range>
-        <noise><type>gaussian</type><mean>0.0</mean><stddev>0.01</stddev></noise>
-      </ray>
-      <plugin name="lidar_plugin" filename="libgazebo_ros_ray_sensor.so">
-        <ros><remapping>~/out:=/scan</remapping></ros>
-        <output_type>sensor_msgs/LaserScan</output_type>
-        <frame_name>lidar_link</frame_name>
-      </plugin>
-    </sensor>
-  </gazebo>
-  <!-- RGB-D Camera -->
-  <gazebo reference="camera_link">
-    <sensor type="depth" name="rgbd_camera">
-      <update_rate>30.0</update_rate>
-      <camera>
-        <horizontal_fov>1.0472</horizontal_fov>
-        <image><width>640</width><height>480</height><format>R8G8B8</format></image>
-        <clip><near>0.1</near><far>10.0</far></clip>
-      </camera>
-      <plugin name="rgbd_plugin" filename="libgazebo_ros_camera.so">
-        <ros>
-          <remapping>~/image_raw:=/camera/image_raw</remapping>
-          <remapping>~/camera_info:=/camera/camera_info</remapping>
-          <remapping>~/depth/image_raw:=/camera/depth/image_raw</remapping>
-          <remapping>~/points:=/camera/points</remapping>
-        </ros>
-        <camera_name>camera</camera_name>
-        <frame_name>camera_optical_frame</frame_name>
-      </plugin>
-    </sensor>
-  </gazebo>
+<?xml version="1.0" encoding="utf-8"?>
+<!-- This URDF was automatically created by SolidWorks to URDF Exporter! Originally created by Stephen Brawner (brawner@gmail.com)
+     Commit Version: 1.6.0-4-g7f85cfe  Build Version: 1.6.7995.38578
+     For more information, please see http://wiki.ros.org/sw_urdf_exporter -->
+<robot
+  name="assembly_of_robot">
+  <link
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