Commit message: fix(simulation_pkg): sync URDF xacro with assembly_of_robot (correct links, joints, Gazebo plugins)

File: ros2_mobile_manipulator_ws/src/simulation_pkg/urdf/mobile_manipulator.urdf.xacro (robot description, xacro)
@@ -1,789 +1,654 @@
 <?xml version="1.0" encoding="utf-8"?>
-<!-- This URDF was automatically created by SolidWorks to URDF Exporter! Originally created by Stephen Brawner (brawner@gmail.com)
-     Commit Version: 1.6.0-4-g7f85cfe  Build Version: 1.6.7995.38578
-     For more information, please see http://wiki.ros.org/sw_urdf_exporter -->
-<robot
-  name="assembly_of_robot">
-  <link
-    name="base_link">
-    <inertial>
-      <origin
-        xyz="-0.00370560542088127 -0.00123891547063168 -0.0326447076903412"
-        rpy="0 0 0" />
-      <mass
-        value="0.0585904996282878" />
-      <inertia
-        ixx="8.00882758728889E-05"
-        ixy="-9.08460677919354E-06"
-        ixz="-4.47145682288692E-13"
-        iyy="0.000258854069540987"
-        iyz="-1.24068479421353E-12"
-        izz="0.000335783016348923" />
-    </inertial>
-    <visual>
-      <origin
-        xyz="0 0 0"
-        rpy="0 0 0" />
-      <geometry>
-        <mesh
-          filename="package://assembly_of_robot/meshes/base_link.STL" />
-      </geometry>
-      <material
-        name="">
-        <color
-          rgba="0.666666666666667 0.698039215686274 0.768627450980392 1" />
-      </material>
-    </visual>
-    <collision>
-      <origin
-        xyz="0 0 0"
-        rpy="0 0 0" />
-      <geometry>
-        <mesh
-          filename="package://assembly_of_robot/meshes/base_link.STL" />
-      </geometry>
-    </collision>
-  </link>
-  <link
-    name="wheel_fl_link">
-    <inertial>
-      <origin
-        xyz="-0.000105669853970536 -0.00174681357516555 0.0101270123724146"
-        rpy="0 0 0" />
-      <mass
-        value="0.166945648341111" />
-      <inertia
-        ixx="6.72961952966562E-05"
-        ixy="8.75460776044797E-10"
-        ixz="3.1755781149978E-12"
-        iyy="6.72928970285414E-05"
-        iyz="1.03915652666965E-12"
-        izz="0.000113206411676655" />
-    </inertial>
-    <visual>
-      <origin
-        xyz="0 0 0"
-        rpy="0 0 0" />
-      <geometry>
-        <mesh
-          filename="package://assembly_of_robot/meshes/wheel_fl_link.STL" />
-      </geometry>
-      <material
-        name="">
-        <color
-          rgba="0.792156862745098 0.819607843137255 0.933333333333333 1" />
-      </material>
-    </visual>
-    <collision>
-      <origin
-        xyz="0 0 0"
-        rpy="0 0 0" />
-      <geometry>
-        <mesh
-          filename="package://assembly_of_robot/meshes/wheel_fl_link.STL" />
-      </geometry>
-    </collision>
-  </link>
-  <joint
-    name="wheel_fl_joint"
-    type="fixed">
-    <origin
-      xyz="-0.064799 -0.06515 -0.020884"
-      rpy="1.5708 -0.060409 0.050643" />
-    <parent
-      link="base_link" />
-    <child
-      link="wheel_fl_link" />
-    <axis
-      xyz="0 0 0" />
-  </joint>
-  <link
-    name="wheel_fr_link">
-    <inertial>
-      <origin
-        xyz="-0.000105670029036942 0.00174681288738787 0.010127012388173"
-        rpy="0 0 0" />
-      <mass
-        value="0.166945648268322" />
-      <inertia
-        ixx="6.72959886592619E-05"
-        ixy="-1.18547893310603E-09"
-        ixz="3.06215474412157E-12"
-        iyy="6.72931038073597E-05"
-        iyz="-9.2618000400134E-13"
-        izz="0.000113206411590483" />
-    </inertial>
-    <visual>
-      <origin
-        xyz="0 0 0"
-        rpy="0 0 0" />
-      <geometry>
-        <mesh
-          filename="package://assembly_of_robot/meshes/wheel_fr_link.STL" />
-      </geometry>
-      <material
-        name="">
-        <color
-          rgba="0.792156862745098 0.819607843137255 0.933333333333333 1" />
-      </material>
-    </visual>
-    <collision>
-      <origin
-        xyz="0 0 0"
-        rpy="0 0 0" />
-      <geometry>
-        <mesh
-          filename="package://assembly_of_robot/meshes/wheel_fr_link.STL" />
-      </geometry>
-    </collision>
-  </link>
-  <joint
-    name="wheel_fr_joint"
-    type="fixed">
-    <origin
-      xyz="-0.070948 0.056167 -0.020884"
-      rpy="-1.5708 -0.060409 0.050643" />
-    <parent
-      link="base_link" />
-    <child
-      link="wheel_fr_link" />
-    <axis
-      xyz="0 0 0" />
-  </joint>
-  <link
-    name="wheel_bl_link">
-    <inertial>
-      <origin
-        xyz="-0.000105669853960988 -0.0017468135751744 0.0101270123724197"
-        rpy="0 0 0" />
-      <mass
-        value="0.166945648341348" />
-      <inertia
-        ixx="6.72961952967705E-05"
-        ixy="8.75460791537877E-10"
-        ixz="3.17557931693756E-12"
-        iyy="6.72928970285945E-05"
-        iyz="1.03916985727418E-12"
-        izz="0.000113206411676816" />
-    </inertial>
-    <visual>
-      <origin
-        xyz="0 0 0"
-        rpy="0 0 0" />
-      <geometry>
-        <mesh
-          filename="package://assembly_of_robot/meshes/wheel_bl_link.STL" />
-      </geometry>
-      <material
-        name="">
-        <color
-          rgba="0.792156862745098 0.819607843137255 0.933333333333333 1" />
-      </material>
-    </visual>
-    <collision>
-      <origin
-        xyz="0 0 0"
-        rpy="0 0 0" />
-      <geometry>
-        <mesh
-          filename="package://assembly_of_robot/meshes/wheel_bl_link.STL" />
-      </geometry>
-    </collision>
-  </link>
-  <joint
-    name="wheel_bl_joint"
-    type="fixed">
-    <origin
-      xyz="0.063537 -0.058645 -0.020884"
-      rpy="1.5708 -0.060409 0.050643" />
-    <parent
-      link="base_link" />
-    <child
-      link="wheel_bl_link" />
-    <axis
-      xyz="0 0 0" />
-  </joint>
-  <link
-    name="wheel_br_link">
-    <inertial>
-      <origin
-        xyz="-0.000105670029167615 0.00174681288747511 0.010127012388229"
-        rpy="0 0 0" />
-      <mass
-        value="0.166945648269942" />
-      <inertia
-        ixx="6.72959886593697E-05"
-        ixy="-1.18547871982134E-09"
-        ixz="3.06227103560424E-12"
-        iyy="6.72931038077175E-05"
-        iyz="-9.26253933036976E-13"
-        izz="0.000113206411590851" />
-    </inertial>
-    <visual>
-      <origin
-        xyz="0 0 0"
-        rpy="0 0 0" />
-      <geometry>
-        <mesh
-          filename="package://assembly_of_robot/meshes/wheel_br_link.STL" />
-      </geometry>
-      <material
-        name="">
-        <color
-          rgba="0.792156862745098 0.819607843137255 0.933333333333333 1" />
-      </material>
-    </visual>
-    <collision>
-      <origin
-        xyz="0 0 0"
-        rpy="0 0 0" />
-      <geometry>
-        <mesh
-          filename="package://assembly_of_robot/meshes/wheel_br_link.STL" />
-      </geometry>
-    </collision>
-  </link>
-  <joint
-    name="wheel_br_joint"
-    type="fixed">
-    <origin
-      xyz="0.057387 0.062672 -0.020884"
-      rpy="-1.5708 -0.060409 0.050643" />
-    <parent
-      link="base_link" />
-    <child
-      link="wheel_br_link" />
-    <axis
-      xyz="0 0 0" />
-  </joint>
-  <link
-    name="arm_link_1">
-    <inertial>
-      <origin
-        xyz="-0.124122626261111 0.00674578860620575 -0.0308255459423702"
-        rpy="0 0 0" />
-      <mass
-        value="8.1278852649819E-05" />
-      <inertia
-        ixx="4.93089984265765E-09"
-        ixy="-3.70030615453607E-10"
-        ixz="-6.73001887244955E-11"
-        iyy="2.95256868033253E-10"
-        iyz="5.33829838018978E-12"
-        izz="4.99315942171251E-09" />
-    </inertial>
-    <visual>
-      <origin
-        xyz="0 0 0"
-        rpy="0 0 0" />
-      <geometry>
-        <mesh
-          filename="package://assembly_of_robot/meshes/arm_link_1.STL" />
-      </geometry>
-      <material
-        name="">
-        <color
-          rgba="0.917647058823529 0.917647058823529 0.917647058823529 1" />
-      </material>
-    </visual>
-    <collision>
-      <origin
-        xyz="0 0 0"
-        rpy="0 0 0" />
-      <geometry>
-        <mesh
-          filename="package://assembly_of_robot/meshes/arm_link_1.STL" />
-      </geometry>
-    </collision>
-  </link>
-  <joint
-    name="arm_joint_1"
-    type="fixed">
-    <origin
-      xyz="0.18587 0.0065057 0.10591"
-      rpy="-3.0796 -0.66341 -0.035278" />
-    <parent
-      link="base_link" />
-    <child
-      link="arm_link_1" />
-    <axis
-      xyz="0 0 0" />
-  </joint>
-  <link
-    name="arm_link_2">
-    <inertial>
-      <origin
-        xyz="0.00648574509338751 -0.0035676648492927 0.0146673556846963"
-        rpy="0 0 0" />
-      <mass
-        value="5.57519132003526E-05" />
-      <inertia
-        ixx="1.44807551587359E-09"
-        ixy="4.27495052985691E-10"
-        ixz="-4.51952909781509E-11"
-        iyy="3.63616413413215E-10"
-        iyz="1.30323710094228E-10"
-        izz="1.70581897775778E-09" />
-    </inertial>
-    <visual>
-      <origin
-        xyz="0 0 0"
-        rpy="0 0 0" />
-      <geometry>
-        <mesh
-          filename="package://assembly_of_robot/meshes/arm_link_2.STL" />
-      </geometry>
-      <material
-        name="">
-        <color
-          rgba="0.917647058823529 0.917647058823529 0.917647058823529 1" />
-      </material>
-    </visual>
-    <collision>
-      <origin
-        xyz="0 0 0"
-        rpy="0 0 0" />
-      <geometry>
-        <mesh
-          filename="package://assembly_of_robot/meshes/arm_link_2.STL" />
-      </geometry>
-    </collision>
-  </link>
-  <joint
-    name="arm_joint_2"
-    type="fixed">
-    <origin
-      xyz="-0.0977341582856277 0.032098573245808 -0.0458965624183291"
-      rpy="1.57079632679489 -0.605405747453626 -0.0791549736736961" />
-    <parent
-      link="arm_link_1" />
-    <child
-      link="arm_link_2" />
-    <axis
-      xyz="0 0 0" />
-  </joint>
-  <link
-    name="arm_link_3">
-    <inertial>
-      <origin
-        xyz="0.0018500879530019 0.00214391271618598 0.0146673556846982"
-        rpy="0 0 0" />
-      <mass
-        value="5.57519132003528E-05" />
-      <inertia
-        ixx="7.09211449765935E-10"
-        ixy="6.6189105909767E-10"
-        ixz="1.10556176440161E-10"
-        iyy="1.10248047952088E-09"
-        iyz="-8.24876693224881E-11"
-        izz="1.70581897775779E-09" />
-    </inertial>
-    <visual>
-      <origin
-        xyz="0 0 0"
-        rpy="0 0 0" />
-      <geometry>
-        <mesh
-          filename="package://assembly_of_robot/meshes/arm_link_3.STL" />
-      </geometry>
-      <material
-        name="">
-        <color
-          rgba="0.917647058823529 0.917647058823529 0.917647058823529 1" />
-      </material>
-    </visual>
-    <collision>
-      <origin
-        xyz="0 0 0"
-        rpy="0 0 0" />
-      <geometry>
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