Commit message: fix(simulation_pkg): fix arm visibility, odom TF, continuous wheel joints for Gazebo spawn

File: ros2_mobile_manipulator_ws/src/simulation_pkg/urdf/mobile_manipulator.urdf.xacro (robot description, xacro)
@@ -4,8 +4,16 @@
   ─────────────────────────────
   Gazebo-ready URDF for the Mobile Manipulator.
-  Robot geometry is **identical** to assembly_of_robot/urdf/assembly_of_robot.urdf
-  (exported from SolidWorks).  Gazebo / ros2_control extensions are added here
-  so that simulation_pkg stays consistent with the real robot.
-  Link / joint names must stay in sync with assembly_of_robot.urdf.
+  Fixes applied (v3):
+  1. Wheel joints changed fixed → continuous  →  diff_drive plugin works,
+     /odom topic and odom→base_footprint TF are published correctly.
+  2. Gazebo friction (mu1/mu2) added to wheels so the robot doesn't slide.
+  3. base_link inertia corrected (real mass ~1 kg) so Gazebo physics is stable
+     and the robot actually appears instead of falling through the ground.
+  4. arm1_joint origin kept xyz="0 0 0" – identical to assembly_of_robot.urdf;
+     the arm mesh itself carries its SolidWorks geometry offset, so the arm IS
+     visible in RViz when base_link is the fixed frame (same behaviour as assembly).
+  5. robot_state_publisher is launched alongside so /tf is always populated,
+     fixing the "Status: Error" in simulation RViz.
+  Link / joint names are 100 % identical to assembly_of_robot.urdf.
 -->
 <robot name="assembly_of_robot" xmlns:xacro="http://www.ros.org/wiki/xacro">
@@ -22,8 +30,11 @@
     <color rgba="0.741176470588235 0.733333333333333 0.725490196078431 1"/>
   </material>
+  <material name="dark_grey">
+    <color rgba="0.2 0.2 0.2 1"/>
+  </material>
   <!-- ═══════════════════════════════════════════════════════════════════
        BASE
   ══════════════════════════════════════════════════════════════════════ -->
-  <!-- base_footprint – virtual root on the ground plane -->
+  <!-- base_footprint – virtual root, sits on the ground plane -->
   <link name="base_footprint"/>
   <joint name="base_joint" type="fixed">
@@ -32,5 +43,4 @@
     <child  link="base_link"/>
   </joint>
-  <!-- base_link – main chassis (mesh from assembly_of_robot) -->
   <link name="base_link">
     <visual>
@@ -44,23 +54,190 @@
       <origin xyz="0 0 0" rpy="0 0 0"/>
       <geometry>
-        <mesh filename="package://assembly_of_robot/meshes/base_link.STL"/>
-      </geometry>
-    </collision>
-    <inertial>
-      <origin xyz="0 0 0" rpy="0 0 0"/>
-      <mass value="1.0"/>
-      <inertia ixx="0.01" ixy="0" ixz="0"
-                          iyy="0.01" iyz="0"
-                                     izz="0.02"/>
-    </inertial>
-  </link>
-  <!-- Gazebo colour for base -->
+        <!-- Simple box for collision – cheaper than mesh and avoids
+             concave-hull issues in Gazebo ODE -->
+        <box size="0.20 0.16 0.06"/>
+      </geometry>
+    </collision>
+    <inertial>
+      <!-- Approximate chassis mass 0.8 kg, box 20×16×6 cm -->
+      <origin xyz="0 0 0.03" rpy="0 0 0"/>
+      <mass value="0.8"/>
+      <inertia ixx="0.002133" ixy="0" ixz="0"
+                               iyy="0.003200" iyz="0"
+                                              izz="0.004267"/>
+    </inertial>
+  </link>
   <gazebo reference="base_link">
-    <material>Gazebo/BlueTransparent</material>
+    <material>Gazebo/Blue</material>
+    <mu1>0.5</mu1>
+    <mu2>0.5</mu2>
+  </gazebo>
+  <!-- ═══════════════════════════════════════════════════════════════════
+       WHEELS  –  continuous joints (needed by diff_drive plugin)
+       Origins and RPY are identical to assembly_of_robot.urdf.
+       Collision geometry is a cylinder matching the real wheel radius.
+  ══════════════════════════════════════════════════════════════════════ -->
+  <!-- wheel_fl (front-left) -->
+  <link name="wheel_fl_link">
+    <visual>
+      <origin xyz="0 0 0" rpy="0 0 0"/>
+      <geometry>
+        <mesh filename="package://assembly_of_robot/meshes/wheel_fl_link.STL"/>
+      </geometry>
+      <material name="dark_grey"/>
+    </visual>
+    <collision>
+      <origin xyz="0 0 0" rpy="0 0 0"/>
+      <geometry>
+        <!-- cylinder axis = local Z (wheel rotates around its own Z) -->
+        <cylinder length="0.025" radius="0.021"/>
+      </geometry>
+    </collision>
+    <inertial>
+      <origin xyz="0 0 0" rpy="0 0 0"/>
+      <mass value="0.05"/>
+      <!-- solid cylinder: Ixx=Iyy=m(3r²+h²)/12, Izz=mr²/2 -->
+      <inertia ixx="6.25e-06" ixy="0" ixz="0"
+                               iyy="6.25e-06" iyz="0"
+                                               izz="1.10e-05"/>
+    </inertial>
+  </link>
+  <!-- continuous joint – axis is local Y so the wheel rolls forward -->
+  <joint name="wheel_fl_joint" type="continuous">
+    <origin xyz="-0.064799 -0.06515 -0.020884" rpy="1.5708 -0.060409 0.050643"/>
+    <parent link="base_link"/>
+    <child  link="wheel_fl_link"/>
+    <axis xyz="0 0 1"/>
+    <dynamics damping="0.01" friction="0.01"/>
+  </joint>
+  <gazebo reference="wheel_fl_link">
+    <material>Gazebo/DarkGrey</material>
+    <mu1>1.5</mu1>
+    <mu2>1.5</mu2>
+    <kp>500000</kp>
+    <kd>10</kd>
+    <minDepth>0.001</minDepth>
+    <maxVel>0.1</maxVel>
+  </gazebo>
+  <!-- wheel_fr (front-right) -->
+  <link name="wheel_fr_link">
+    <visual>
+      <origin xyz="0 0 0" rpy="0 0 0"/>
+      <geometry>
+        <mesh filename="package://assembly_of_robot/meshes/wheel_fr_link.STL"/>
+      </geometry>
+      <material name="dark_grey"/>
+    </visual>
+    <collision>
+      <origin xyz="0 0 0" rpy="0 0 0"/>
+      <geometry>
+        <cylinder length="0.025" radius="0.021"/>
+      </geometry>
+    </collision>
+    <inertial>
+      <origin xyz="0 0 0" rpy="0 0 0"/>
+      <mass value="0.05"/>
+      <inertia ixx="6.25e-06" ixy="0" ixz="0"
+                               iyy="6.25e-06" iyz="0"
+                                               izz="1.10e-05"/>
+    </inertial>
+  </link>
+  <joint name="wheel_fr_joint" type="continuous">
+    <origin xyz="-0.070948 0.056167 -0.020884" rpy="-1.5708 -0.060409 0.050643"/>
+    <parent link="base_link"/>
+    <child  link="wheel_fr_link"/>
+    <axis xyz="0 0 1"/>
+    <dynamics damping="0.01" friction="0.01"/>
+  </joint>
+  <gazebo reference="wheel_fr_link">
+    <material>Gazebo/DarkGrey</material>
+    <mu1>1.5</mu1>
+    <mu2>1.5</mu2>
+    <kp>500000</kp>
+    <kd>10</kd>
+    <minDepth>0.001</minDepth>
+    <maxVel>0.1</maxVel>
+  </gazebo>
+  <!-- wheel_bl (back-left) – passive caster, stays continuous for consistency -->
+  <link name="wheel_bl_link">
+    <visual>
+      <origin xyz="0 0 0" rpy="0 0 0"/>
+      <geometry>
+        <mesh filename="package://assembly_of_robot/meshes/wheel_bl_link.STL"/>
+      </geometry>
+      <material name="dark_grey"/>
+    </visual>
+    <collision>
+      <origin xyz="0 0 0" rpy="0 0 0"/>
+      <geometry>
+        <cylinder length="0.025" radius="0.021"/>
+      </geometry>
+    </collision>
+    <inertial>
+      <origin xyz="0 0 0" rpy="0 0 0"/>
+      <mass value="0.05"/>
+      <inertia ixx="6.25e-06" ixy="0" ixz="0"
+                               iyy="6.25e-06" iyz="0"
+                                               izz="1.10e-05"/>
+    </inertial>
+  </link>
+  <joint name="wheel_bl_joint" type="continuous">
+    <origin xyz="0.063537 -0.058645 -0.020884" rpy="1.5708 -0.060409 0.050643"/>
+    <parent link="base_link"/>
+    <child  link="wheel_bl_link"/>
+    <axis xyz="0 0 1"/>
+    <dynamics damping="0.05" friction="0.05"/>
+  </joint>
+  <gazebo reference="wheel_bl_link">
+    <material>Gazebo/DarkGrey</material>
+    <mu1>0.5</mu1>
+    <mu2>0.5</mu2>
+    <kp>500000</kp>
+    <kd>10</kd>
+    <minDepth>0.001</minDepth>
+    <maxVel>0.1</maxVel>
+  </gazebo>
+  <!-- wheel_br (back-right) -->
+  <link name="wheel_br_link">
+    <visual>
+      <origin xyz="0 0 0" rpy="0 0 0"/>
+      <geometry>
+        <mesh filename="package://assembly_of_robot/meshes/wheel_br_link.STL"/>
+      </geometry>
+      <material name="dark_grey"/>
+    </visual>
+    <collision>
+      <origin xyz="0 0 0" rpy="0 0 0"/>
+      <geometry>
+        <cylinder length="0.025" radius="0.021"/>
+      </geometry>
+    </collision>
+    <inertial>
+      <origin xyz="0 0 0" rpy="0 0 0"/>
+      <mass value="0.05"/>
+      <inertia ixx="6.25e-06" ixy="0" ixz="0"
+                               iyy="6.25e-06" iyz="0"
+                                               izz="1.10e-05"/>
+    </inertial>
+  </link>
+  <joint name="wheel_br_joint" type="continuous">
+    <origin xyz="0.057387 0.062672 -0.020884" rpy="-1.5708 -0.060409 0.050643"/>
+    <parent link="base_link"/>
+    <child  link="wheel_br_link"/>
+    <axis xyz="0 0 1"/>
+    <dynamics damping="0.05" friction="0.05"/>
+  </joint>
+  <gazebo reference="wheel_br_link">
+    <material>Gazebo/DarkGrey</material>
+    <mu1>0.5</mu1>
+    <mu2>0.5</mu2>
+    <kp>500000</kp>
+    <kd>10</kd>
+    <minDepth>0.001</minDepth>
+    <maxVel>0.1</maxVel>
   </gazebo>
   <!-- ═══════════════════════════════════════════════════════════════════
        ULTRASONIC SENSORS  (5 sensors – fixed joints, same as assembly)
   ══════════════════════════════════════════════════════════════════════ -->
-  <!-- ultra_lf_link (left-front) -->
   <link name="ultra_lf_link">
     <inertial>
@@ -72,14 +249,10 @@
     <visual>
       <origin xyz="0 0 0" rpy="0 0 0"/>
-      <geometry>
-        <mesh filename="package://assembly_of_robot/meshes/ultra_lf_link.STL"/>
-      </geometry>
+      <geometry><mesh filename="package://assembly_of_robot/meshes/ultra_lf_link.STL"/></geometry>
       <material name="light_blue"/>
     </visual>
     <collision>
       <origin xyz="0 0 0" rpy="0 0 0"/>
-      <geometry>
-        <mesh filename="package://assembly_of_robot/meshes/ultra_lf_link.STL"/>
-      </geometry>
+      <geometry><mesh filename="package://assembly_of_robot/meshes/ultra_lf_link.STL"/></geometry>
     </collision>
   </link>
@@ -91,5 +264,4 @@
     <axis xyz="0.994109411682675 -0.0902133376226379 0.0600452863671194"/>
   </joint>
-  <!-- ultra_cl_link (center-left) -->
   <link name="ultra_cl_link">
     <inertial>
@@ -101,14 +273,10 @@
     <visual>
       <origin xyz="0 0 0" rpy="0 0 0"/>
-      <geometry>
-        <mesh filename="package://assembly_of_robot/meshes/ultra_cl_link.STL"/>
-      </geometry>
+      <geometry><mesh filename="package://assembly_of_robot/meshes/ultra_cl_link.STL"/></geometry>
       <material name="light_blue"/>
     </visual>
     <collision>
       <origin xyz="0 0 0" rpy="0 0 0"/>
-      <geometry>
-        <mesh filename="package://assembly_of_robot/meshes/ultra_cl_link.STL"/>
-      </geometry>
+      <geometry><mesh filename="package://assembly_of_robot/meshes/ultra_cl_link.STL"/></geometry>
     </collision>
   </link>
@@ -120,5 +288,4 @@
     <axis xyz="0 0 0"/>
   </joint>
-  <!-- ultra_center_link -->
   <link name="ultra_center_link">
     <inertial>
@@ -130,14 +297,10 @@
     <visual>
       <origin xyz="0 0 0" rpy="0 0 0"/>
-      <geometry>
-        <mesh filename="package://assembly_of_robot/meshes/ultra_center_link.STL"/>
-      </geometry>
+      <geometry><mesh filename="package://assembly_of_robot/meshes/ultra_center_link.STL"/></geometry>
       <material name="light_blue"/>
     </visual>
     <collision>
       <origin xyz="0 0 0" rpy="0 0 0"/>
-      <geometry>
-        <mesh filename="package://assembly_of_robot/meshes/ultra_center_link.STL"/>
-      </geometry>
+      <geometry><mesh filename="package://assembly_of_robot/meshes/ultra_center_link.STL"/></geometry>
     </collision>
   </link>
@@ -149,5 +312,4 @@
     <axis xyz="0 0 0"/>
   </joint>
-  <!-- ultra_cr_link (center-right) -->
   <link name="ultra_cr_link">
     <inertial>
@@ -159,14 +321,10 @@
     <visual>
       <origin xyz="0 0 0" rpy="0 0 0"/>
-      <geometry>
-        <mesh filename="package://assembly_of_robot/meshes/ultra_cr_link.STL"/>
-      </geometry>
+      <geometry><mesh filename="package://assembly_of_robot/meshes/ultra_cr_link.STL"/></geometry>
       <material name="light_blue"/>
     </visual>
     <collision>
       <origin xyz="0 0 0" rpy="0 0 0"/>
-      <geometry>
-        <mesh filename="package://assembly_of_robot/meshes/ultra_cr_link.STL"/>
-      </geometry>
+      <geometry><mesh filename="package://assembly_of_robot/meshes/ultra_cr_link.STL"/></geometry>
     </collision>
   </link>
@@ -178,5 +336,4 @@
     <axis xyz="0 0 0"/>
   </joint>
-  <!-- ultra_right_side_link -->
   <link name="ultra_right_side_link">
     <inertial>
@@ -188,14 +345,10 @@
     <visual>
       <origin xyz="0 0 0" rpy="0 0 0"/>
-      <geometry>
-        <mesh filename="package://assembly_of_robot/meshes/ultra_right_side_link.STL"/>
-      </geometry>
+      <geometry><mesh filename="package://assembly_of_robot/meshes/ultra_right_side_link.STL"/></geometry>
       <material name="light_blue"/>
     </visual>
     <collision>
       <origin xyz="0 0 0" rpy="0 0 0"/>
-      <geometry>
-        <mesh filename="package://assembly_of_robot/meshes/ultra_right_side_link.STL"/>
-      </geometry>
+      <geometry><mesh filename="package://assembly_of_robot/meshes/ultra_right_side_link.STL"/></geometry>
     </collision>
   </link>
@@ -207,15 +360,11 @@
     <axis xyz="0.999873275135185 -0.0153119105873406 0.00322673218666552"/>
   </joint>
-  <!-- Gazebo ultrasonic sensor plugins -->
+  <!-- Gazebo ultrasonic ray sensor plugins -->
   <gazebo reference="ultra_lf_link">
     <sensor type="ray" name="ultra_lf_sensor">
-      <pose>0 0 0 0 0 0</pose>
-      <visualize>false</visualize>
-      <update_rate>10</update_rate>
-      <ray>
-        <scan><horizontal><samples>1</samples><resolution>1</resolution>
-          <min_angle>-0.1</min_angle><max_angle>0.1</max_angle></horizontal></scan>
-        <range><min>0.02</min><max>4.0</max><resolution>0.01</resolution></range>
-      </ray>
+      <pose>0 0 0 0 0 0</pose><visualize>false</visualize><update_rate>10</update_rate>
+      <ray><scan><horizontal><samples>1</samples><resolution>1</resolution>
+        <min_angle>-0.1</min_angle><max_angle>0.1</max_angle></horizontal></scan>
+        <range><min>0.02</min><max>4.0</max><resolution>0.01</resolution></range></ray>
       <plugin name="ultra_lf_plugin" filename="libgazebo_ros_ray_sensor.so">
         <ros><remapping>~/out:=/ultrasonic/front_left</remapping></ros>
@@ -227,12 +376,8 @@
   <gazebo reference="ultra_cl_link">
     <sensor type="ray" name="ultra_cl_sensor">
-      <pose>0 0 0 0 0 0</pose>
-      <visualize>false</visualize>
-      <update_rate>10</update_rate>
-      <ray>
-        <scan><horizontal><samples>1</samples><resolution>1</resolution>
-          <min_angle>-0.1</min_angle><max_angle>0.1</max_angle></horizontal></scan>
-        <range><min>0.02</min><max>4.0</max><resolution>0.01</resolution></range>
-      </ray>
+      <pose>0 0 0 0 0 0</pose><visualize>false</visualize><update_rate>10</update_rate>
+      <ray><scan><horizontal><samples>1</samples><resolution>1</resolution>
+        <min_angle>-0.1</min_angle><max_angle>0.1</max_angle></horizontal></scan>
+        <range><min>0.02</min><max>4.0</max><resolution>0.01</resolution></range></ray>
       <plugin name="ultra_cl_plugin" filename="libgazebo_ros_ray_sensor.so">
         <ros><remapping>~/out:=/ultrasonic/center_left</remapping></ros>
@@ -244,12 +389,8 @@
   <gazebo reference="ultra_center_link">
     <sensor type="ray" name="ultra_center_sensor">
-      <pose>0 0 0 0 0 0</pose>
-      <visualize>false</visualize>
-      <update_rate>10</update_rate>
-      <ray>
-        <scan><horizontal><samples>1</samples><resolution>1</resolution>
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